Commit message: feat(stage2): validate vehicle simulation and sensor runtime

File: starter_ws/src/sanitation_vehicle_description/urdf/sanitation_vehicle.urdf.xacro (robot description, xacro)
@@ -2,10 +2,5 @@
 <robot name="sanitation_vehicle" xmlns:xacro="http://ros.org/wiki/xacro">
   <!-- Reuse maintained Linorobot2 macros without modifying upstream source. -->
-  <xacro:include filename="$(find linorobot2_description)/urdf/mech/base.urdf.xacro"/>
-  <xacro:include filename="$(find linorobot2_description)/urdf/mech/wheel.urdf.xacro"/>
-  <xacro:include filename="$(find linorobot2_description)/urdf/sensors/plugins.urdf.xacro"/>
   <xacro:include filename="$(find linorobot2_description)/urdf/sensors/imu.urdf.xacro"/>
-  <xacro:include filename="$(find linorobot2_description)/urdf/sensors/generic_laser.urdf.xacro"/>
-  <xacro:include filename="$(find linorobot2_description)/urdf/sensors/depth_sensor.urdf.xacro"/>
   <xacro:include filename="$(find linorobot2_description)/urdf/controllers/skid_steer.urdf.xacro"/>
   <!-- Baseline geometry; replace with measured real vehicle values later. -->
@@ -21,32 +16,148 @@
   <xacro:property name="wheel_mass" value="3.0"/>
   <xacro:property name="cleaning_width" value="0.65"/>
-  <xacro:base
-    length="${base_length}"
-    width="${base_width}"
-    height="${base_height}"
-    mass="${base_mass}"
-    wheel_radius="${wheel_radius}"
-    wheel_pos_z="${wheel_pos_z}"
-    mesh_file=""
-  />
-  <xacro:wheel side="front_left" radius="${wheel_radius}" width="${wheel_width}"
-    pos_x="${wheel_pos_x}" pos_y="${wheel_pos_y}" pos_z="${wheel_pos_z}"
-    mass="${wheel_mass}" mesh_file=""/>
-  <xacro:wheel side="front_right" radius="${wheel_radius}" width="${wheel_width}"
-    pos_x="${wheel_pos_x}" pos_y="${-wheel_pos_y}" pos_z="${wheel_pos_z}"
-    mass="${wheel_mass}" mesh_file=""/>
-  <xacro:wheel side="rear_left" radius="${wheel_radius}" width="${wheel_width}"
-    pos_x="${-wheel_pos_x}" pos_y="${wheel_pos_y}" pos_z="${wheel_pos_z}"
-    mass="${wheel_mass}" mesh_file=""/>
-  <xacro:wheel side="rear_right" radius="${wheel_radius}" width="${wheel_width}"
-    pos_x="${-wheel_pos_x}" pos_y="${-wheel_pos_y}" pos_z="${wheel_pos_z}"
-    mass="${wheel_mass}" mesh_file=""/>
+  <!-- Local primitive chassis avoids the upstream Gazebo-classic visual
+       override colliding with URDF materials in Ogre2 / Gazebo Harmonic. -->
+  <link name="base_footprint"/>
+  <link name="base_link">
+    <visual>
+      <geometry><box size="${base_length} ${base_width} ${base_height}"/></geometry>
+      <material name="sanitation_chassis_yellow">
+        <color rgba="0.84 0.63 0.05 1.0"/>
+      </material>
+    </visual>
+    <collision>
+      <geometry><box size="${base_length} ${base_width} ${base_height}"/></geometry>
+    </collision>
+    <inertial>
+      <mass value="${base_mass}"/>
+      <inertia
+        ixx="${(base_mass / 12.0) * (base_width**2 + base_height**2)}"
+        ixy="0" ixz="0"
+        iyy="${(base_mass / 12.0) * (base_length**2 + base_height**2)}"
+        iyz="0"
+        izz="${(base_mass / 12.0) * (base_length**2 + base_width**2)}"/>
+    </inertial>
+  </link>
+  <joint name="base_to_footprint" type="fixed">
+    <parent link="base_footprint"/>
+    <child link="base_link"/>
+    <origin xyz="0 0 ${wheel_radius - wheel_pos_z}" rpy="0 0 0"/>
+  </joint>
+  <xacro:macro name="sanitation_wheel" params="side pos_x pos_y red green blue">
+    <link name="${side}_wheel_link">
+      <visual>
+        <origin rpy="${pi / 2.0} 0 0"/>
+        <geometry><cylinder radius="${wheel_radius}" length="${wheel_width}"/></geometry>
+        <material name="${side}_wheel_material">
+          <color rgba="${red} ${green} ${blue} 1.0"/>
+        </material>
+      </visual>
+      <collision>
+        <origin rpy="${pi / 2.0} 0 0"/>
+        <geometry><cylinder radius="${wheel_radius}" length="${wheel_width}"/></geometry>
+      </collision>
+      <inertial>
+        <mass value="${wheel_mass}"/>
+        <inertia
+          ixx="${(wheel_mass / 12.0) * (3.0 * wheel_radius**2 + wheel_width**2)}"
+          ixy="0" ixz="0"
+          iyy="${0.5 * wheel_mass * wheel_radius**2}"
+          iyz="0"
+          izz="${(wheel_mass / 12.0) * (3.0 * wheel_radius**2 + wheel_width**2)}"/>
+      </inertial>
+    </link>
+    <joint name="${side}_wheel_joint" type="continuous">
+      <axis xyz="0 1 0"/>
+      <parent link="base_link"/>
+      <child link="${side}_wheel_link"/>
+      <origin xyz="${pos_x} ${pos_y} ${wheel_pos_z}" rpy="0 0 0"/>
+    </joint>
+  </xacro:macro>
+  <xacro:sanitation_wheel side="front_left" pos_x="${wheel_pos_x}" pos_y="${wheel_pos_y}"
+    red="0.12" green="0.32" blue="0.62"/>
+  <xacro:sanitation_wheel side="front_right" pos_x="${wheel_pos_x}" pos_y="${-wheel_pos_y}"
+    red="0.13" green="0.33" blue="0.63"/>
+  <xacro:sanitation_wheel side="rear_left" pos_x="${-wheel_pos_x}" pos_y="${wheel_pos_y}"
+    red="0.14" green="0.34" blue="0.64"/>
+  <xacro:sanitation_wheel side="rear_right" pos_x="${-wheel_pos_x}" pos_y="${-wheel_pos_y}"
+    red="0.15" green="0.35" blue="0.65"/>
   <xacro:imu/>
-  <xacro:generic_laser>
+  <link name="laser">
+    <visual>
+      <geometry><cylinder radius="0.045" length="0.06"/></geometry>
+      <material name="sanitation_lidar_green"><color rgba="0.02 0.55 0.20 1.0"/></material>
+    </visual>
+    <collision><geometry><cylinder radius="0.045" length="0.06"/></geometry></collision>
+    <inertial>
+      <mass value="0.1"/>
+      <inertia ixx="0.00006" ixy="0" ixz="0" iyy="0.00006" iyz="0" izz="0.00010"/>
+    </inertial>
+  </link>
+  <joint name="laser_to_base_link" type="fixed">
+    <parent link="base_link"/>
+    <child link="laser"/>
     <origin xyz="0.12 0 0.48" rpy="0 0 0"/>
-  </xacro:generic_laser>
-  <xacro:depth_sensor>
+  </joint>
+  <gazebo reference="laser">
+    <sensor name="sanitation_gpu_lidar" type="gpu_lidar">
+      <topic>scan</topic>
+      <update_rate>10</update_rate>
+      <always_on>true</always_on>
+      <visualize>true</visualize>
+      <lidar>
+        <scan>
+          <horizontal>
+            <samples>360</samples>
+            <resolution>1</resolution>
+            <min_angle>-3.1416</min_angle>
+            <max_angle>3.1416</max_angle>
+          </horizontal>
+          <vertical>
+            <samples>1</samples>
+            <resolution>1</resolution>
+            <min_angle>0.0</min_angle>
+            <max_angle>0.0</max_angle>
+          </vertical>
+        </scan>
+        <range><min>0.08</min><max>12.0</max><resolution>0.01</resolution></range>
+      </lidar>
+    </sensor>
+  </gazebo>
+  <link name="camera_link">
+    <visual>
+      <geometry><box size="0.05 0.14 0.05"/></geometry>
+      <material name="sanitation_camera_red"><color rgba="0.45 0.05 0.05 1.0"/></material>
+    </visual>
+    <collision><geometry><box size="0.05 0.14 0.05"/></geometry></collision>
+    <inertial>
+      <mass value="0.135"/>
+      <inertia ixx="0.00025" ixy="0" ixz="0" iyy="0.00006" iyz="0" izz="0.00025"/>
+    </inertial>
+  </link>
+  <joint name="camera_to_base_link" type="fixed">
+    <parent link="base_link"/>
+    <child link="camera_link"/>
     <origin xyz="0.53 0 0.22" rpy="0 0 0"/>
-  </xacro:depth_sensor>
+  </joint>
+  <link name="camera_depth_link"/>
+  <joint name="camera_depth_joint" type="fixed">
+    <parent link="camera_link"/>
+    <child link="camera_depth_link"/>
+    <origin xyz="0 0 0" rpy="0 0 0"/>
+  </joint>
+  <gazebo reference="camera_link">
+    <sensor name="sanitation_rgbd_camera" type="rgbd_camera">
+      <topic>camera</topic>
+      <update_rate>15</update_rate>
+      <always_on>true</always_on>
+      <visualize>true</visualize>
+      <camera>
+        <optical_frame_id>camera_depth_link</optical_frame_id>
+        <horizontal_fov>1.50098</horizontal_fov>
+        <image><width>640</width><height>480</height><format>R8G8B8</format></image>
+        <clip><near>0.3</near><far>100</far></clip>
+      </camera>
+    </sensor>
+  </gazebo>
   <xacro:diff_drive_controller
     wheel_separation="${wheel_pos_y * 2.0}"
@@ -79,5 +190,5 @@
     <visual>
       <geometry><cylinder radius="0.14" length="0.03"/></geometry>
-      <material name="brush_dark"><color rgba="0.08 0.08 0.08 1.0"/></material>
+      <material name="left_brush_dark"><color rgba="0.08 0.08 0.08 1.0"/></material>
     </visual>
     <collision><geometry><cylinder radius="0.14" length="0.03"/></geometry></collision>
@@ -95,5 +206,5 @@
     <visual>
       <geometry><cylinder radius="0.14" length="0.03"/></geometry>
-      <material name="brush_dark"/>
+      <material name="right_brush_dark"><color rgba="0.09 0.09 0.09 1.0"/></material>
     </visual>
     <collision><geometry><cylinder radius="0.14" length="0.03"/></geometry></collision>
@@ -128,6 +239,3 @@
     <origin xyz="0.10 0 0.32" rpy="0 0 0"/>
   </joint>
-  <gazebo reference="cleaning_footprint_link">
-    <transparency>0.82</transparency>
-  </gazebo>
 </robot>

Commit message: feat: add Stage4S motion calibration evidence

File: starter_ws/src/sanitation_vehicle_description/urdf/sanitation_vehicle.urdf.xacro (robot description, xacro)
@@ -4,4 +4,15 @@
   <xacro:include filename="$(find linorobot2_description)/urdf/sensors/imu.urdf.xacro"/>
   <xacro:include filename="$(find linorobot2_description)/urdf/controllers/skid_steer.urdf.xacro"/>
+  <!-- Stage4S separates physical geometry from the DiffDrive estimator / command
+       model. Defaults reproduce the Stage4R vehicle exactly. -->
+  <xacro:arg name="physical_wheel_radius" default="0.14"/>
+  <xacro:arg name="physical_track_width" default="0.80"/>
+  <xacro:arg name="drive_wheel_radius" default="0.14"/>
+  <xacro:arg name="drive_wheel_separation" default="0.80"/>
+  <xacro:arg name="wheel_mu_longitudinal" default="1.0"/>
+  <xacro:arg name="wheel_mu_lateral" default="1.0"/>
+  <xacro:arg name="slip_compliance_longitudinal" default="0.0"/>
+  <xacro:arg name="slip_compliance_lateral" default="0.0"/>
+  <xacro:arg name="enable_wheel_slip" default="false"/>
   <!-- Baseline geometry; replace with measured real vehicle values later. -->
   <xacro:property name="base_length" value="1.15"/>
@@ -9,8 +20,15 @@
   <xacro:property name="base_height" value="0.28"/>
   <xacro:property name="base_mass" value="80.0"/>
-  <xacro:property name="wheel_radius" value="0.14"/>
+  <xacro:property name="physical_wheel_radius" value="$(arg physical_wheel_radius)"/>
+  <xacro:property name="physical_track_width" value="$(arg physical_track_width)"/>
+  <xacro:property name="drive_wheel_radius" value="$(arg drive_wheel_radius)"/>
+  <xacro:property name="drive_wheel_separation" value="$(arg drive_wheel_separation)"/>
+  <xacro:property name="wheel_mu_longitudinal" value="$(arg wheel_mu_longitudinal)"/>
+  <xacro:property name="wheel_mu_lateral" value="$(arg wheel_mu_lateral)"/>
+  <xacro:property name="slip_compliance_longitudinal" value="$(arg slip_compliance_longitudinal)"/>
+  <xacro:property name="slip_compliance_lateral" value="$(arg slip_compliance_lateral)"/>
   <xacro:property name="wheel_width" value="0.08"/>
   <xacro:property name="wheel_pos_x" value="0.38"/>
-  <xacro:property name="wheel_pos_y" value="0.40"/>
+  <xacro:property name="wheel_pos_y" value="${physical_track_width / 2.0}"/>
   <xacro:property name="wheel_pos_z" value="-0.02"/>
   <xacro:property name="wheel_mass" value="3.0"/>
@@ -42,5 +60,5 @@
     <parent link="base_footprint"/>
     <child link="base_link"/>
-    <origin xyz="0 0 ${wheel_radius - wheel_pos_z}" rpy="0 0 0"/>
+    <origin xyz="0 0 ${physical_wheel_radius - wheel_pos_z}" rpy="0 0 0"/>
   </joint>
   <xacro:macro name="sanitation_wheel" params="side pos_x pos_y red green blue">
@@ -48,5 +66,5 @@
       <visual>
         <origin rpy="${pi / 2.0} 0 0"/>
-        <geometry><cylinder radius="${wheel_radius}" length="${wheel_width}"/></geometry>
+        <geometry><cylinder radius="${physical_wheel_radius}" length="${wheel_width}"/></geometry>
         <material name="${side}_wheel_material">
           <color rgba="${red} ${green} ${blue} 1.0"/>
@@ -55,14 +73,14 @@
       <collision>
         <origin rpy="${pi / 2.0} 0 0"/>
-        <geometry><cylinder radius="${wheel_radius}" length="${wheel_width}"/></geometry>
+        <geometry><cylinder radius="${physical_wheel_radius}" length="${wheel_width}"/></geometry>
       </collision>
       <inertial>
         <mass value="${wheel_mass}"/>
         <inertia
-          ixx="${(wheel_mass / 12.0) * (3.0 * wheel_radius**2 + wheel_width**2)}"
+          ixx="${(wheel_mass / 12.0) * (3.0 * physical_wheel_radius**2 + wheel_width**2)}"
           ixy="0" ixz="0"
-          iyy="${0.5 * wheel_mass * wheel_radius**2}"
+          iyy="${0.5 * wheel_mass * physical_wheel_radius**2}"
           iyz="0"
-          izz="${(wheel_mass / 12.0) * (3.0 * wheel_radius**2 + wheel_width**2)}"/>
+          izz="${(wheel_mass / 12.0) * (3.0 * physical_wheel_radius**2 + wheel_width**2)}"/>
       </inertial>
     </link>
@@ -73,4 +91,8 @@
       <origin xyz="${pos_x} ${pos_y} ${wheel_pos_z}" rpy="0 0 0"/>
     </joint>
+    <gazebo reference="${side}_wheel_link">
+      <mu1>${wheel_mu_longitudinal}</mu1>
+      <mu2>${wheel_mu_lateral}</mu2>
+    </gazebo>
   </xacro:macro>
   <xacro:sanitation_wheel side="front_left" pos_x="${wheel_pos_x}" pos_y="${wheel_pos_y}"
@@ -161,7 +183,42 @@
   </gazebo>
   <xacro:diff_drive_controller
-    wheel_separation="${wheel_pos_y * 2.0}"
-    wheel_radius="${wheel_radius}"
+    wheel_separation="${drive_wheel_separation}"
+    wheel_radius="${drive_wheel_radius}"
   />
+  <!-- Disabled by default so the split-parameter baseline exactly preserves
+       Stage4R contact behavior. It is enabled only for an explicit slip scan. -->
+  <xacro:if value="$(arg enable_wheel_slip)">
+    <gazebo>
+      <plugin filename="gz-sim-wheel-slip-system" name="gz::sim::systems::WheelSlip">
+        <xacro:macro name="slip_wheel" params="link_name">
+          <wheel link_name="${link_name}">
+            <wheel_radius>${physical_wheel_radius}</wheel_radius>
+            <slip_compliance_lateral>${slip_compliance_lateral}</slip_compliance_lateral>
+            <slip_compliance_longitudinal>${slip_compliance_longitudinal}</slip_compliance_longitudinal>
+            <wheel_normal_force>250.0</wheel_normal_force>
+          </wheel>
+        </xacro:macro>
+        <xacro:slip_wheel link_name="front_left_wheel_link"/>
+        <xacro:slip_wheel link_name="front_right_wheel_link"/>
+        <xacro:slip_wheel link_name="rear_left_wheel_link"/>
+        <xacro:slip_wheel link_name="rear_right_wheel_link"/>
+      </plugin>
+    </gazebo>
+  </xacro:if>
+  <!-- Model-scoped Gazebo truth. Unlike the world Pose_V bridge, this topic
+       has one producer bound to this model and preserves an explicit frame
+       identity all the way into ROS. It is evaluation-only and must never be
+       fused into the realistic odometry / localization lane. -->
+  <gazebo>
+    <plugin
+      filename="gz-sim-odometry-publisher-system"
+      name="gz::sim::systems::OdometryPublisher">
+      <odom_publish_frequency>50</odom_publish_frequency>
+      <odom_topic>/ground_truth/model_odom_raw</odom_topic>
+      <odom_frame>world</odom_frame>
+      <robot_base_frame>sanitation_vehicle/base_footprint</robot_base_frame>
+      <dimensions>2</dimensions>
+    </plugin>
+  </gazebo>
   <!-- 40 L bin: 0.50 * 0.40 * 0.20 = 0.040 m^3. -->
   <link name="dust_bin_link">

Commit message: complete Stage4U localization evidence

File: starter_ws/src/sanitation_vehicle_description/urdf/sanitation_vehicle.urdf.xacro (robot description, xacro)
@@ -15,4 +15,6 @@
   <xacro:arg name="slip_compliance_lateral" default="0.0"/>
   <xacro:arg name="enable_wheel_slip" default="false"/>
+  <xacro:arg name="lidar_samples" default="360"/>
+  <xacro:arg name="lidar_update_rate" default="10"/>
   <!-- Baseline geometry; replace with measured real vehicle values later. -->
   <xacro:property name="base_length" value="1.15"/>
@@ -34,4 +36,6 @@
   <xacro:property name="wheel_mass" value="3.0"/>
   <xacro:property name="cleaning_width" value="0.65"/>
+  <xacro:property name="lidar_samples" value="$(arg lidar_samples)"/>
+  <xacro:property name="lidar_update_rate" value="$(arg lidar_update_rate)"/>
   <!-- Local primitive chassis avoids the upstream Gazebo-classic visual
        override colliding with URDF materials in Ogre2 / Gazebo Harmonic. -->
@@ -124,5 +128,5 @@
     <sensor name="sanitation_gpu_lidar" type="gpu_lidar">
       <topic>scan</topic>
-      <update_rate>10</update_rate>
+      <update_rate>${lidar_update_rate}</update_rate>
       <always_on>true</always_on>
       <visualize>true</visualize>
@@ -130,5 +134,5 @@
         <scan>
           <horizontal>
-            <samples>360</samples>
+            <samples>${lidar_samples}</samples>
             <resolution>1</resolution>
             <min_angle>-3.1416</min_angle>

Commit message: advance Stage5BR4 active perception

File: starter_ws/src/sanitation_vehicle_description/urdf/sanitation_vehicle.urdf.xacro (robot description, xacro)
@@ -19,4 +19,17 @@
   <!-- Offline G2 capture only. Production launch never overrides this false default. -->
   <xacro:arg name="enable_training_gt" default="false"/>
+  <!-- Stage5BR4 camera ablation. Defaults are the frozen C0 production candidate. -->
+  <xacro:arg name="camera_x" default="0.53"/>
+  <xacro:arg name="camera_y" default="0.0"/>
+  <xacro:arg name="camera_z" default="0.22"/>
+  <xacro:arg name="camera_pitch_rad" default="0.0"/>
+  <xacro:arg name="enable_verification_camera" default="false"/>
+  <xacro:arg name="enable_self_mask_gt" default="false"/>
+  <xacro:arg name="verification_camera_x" default="0.30"/>
+  <xacro:arg name="verification_camera_y" default="0.0"/>
+  <xacro:arg name="verification_camera_z" default="0.70"/>
+  <!-- Gazebo camera optical +X needs positive URDF Y rotation to look down;
+       the external camera spec continues to report conventional negative pitch. -->
+  <xacro:arg name="verification_camera_pitch_rad" default="0.7853981634"/>
   <!-- Baseline geometry; replace with measured real vehicle values later. -->
   <xacro:property name="base_length" value="1.15"/>
@@ -166,5 +179,5 @@
     <parent link="base_link"/>
     <child link="camera_link"/>
-    <origin xyz="0.53 0 0.22" rpy="0 0 0"/>
+    <origin xyz="$(arg camera_x) $(arg camera_y) $(arg camera_z)" rpy="0 $(arg camera_pitch_rad) 0"/>
   </joint>
   <link name="camera_depth_link"/>
@@ -216,4 +229,55 @@
     </xacro:if>
   </gazebo>
+  <!-- C3 verification camera. It is physically and topically independent of
+       the forward discovery camera and is absent from the production default. -->
+  <xacro:if value="$(arg enable_verification_camera)">
+    <link name="verification_camera_link">
+      <visual>
+        <geometry><box size="0.05 0.14 0.05"/></geometry>
+        <material name="sanitation_verification_camera_blue"><color rgba="0.05 0.18 0.55 1.0"/></material>
+      </visual>
+      <collision><geometry><box size="0.05 0.14 0.05"/></geometry></collision>
+      <inertial>
+        <mass value="0.135"/>
+        <inertia ixx="0.00025" ixy="0" ixz="0" iyy="0.00006" iyz="0" izz="0.00025"/>
+      </inertial>
+    </link>
+    <joint name="verification_camera_to_base_link" type="fixed">
+      <parent link="base_link"/>
+      <child link="verification_camera_link"/>
+      <origin xyz="$(arg verification_camera_x) $(arg verification_camera_y) $(arg verification_camera_z)"
+              rpy="0 $(arg verification_camera_pitch_rad) 0"/>
+    </joint>
+    <link name="verification_camera_depth_link"/>
+    <joint name="verification_camera_depth_joint" type="fixed">
+      <parent link="verification_camera_link"/>
+      <child link="verification_camera_depth_link"/>
+      <origin xyz="0 0 0" rpy="0 0 0"/>
+    </joint>
+    <gazebo reference="verification_camera_link">
+      <sensor name="sanitation_verification_rgbd_camera" type="rgbd_camera">
+        <topic>verification_camera</topic>
+        <update_rate>15</update_rate><always_on>true</always_on><visualize>true</visualize>
+        <camera>
+          <optical_frame_id>verification_camera_depth_link</optical_frame_id>
+          <horizontal_fov>1.50098</horizontal_fov>
+          <image><width>640</width><height>480</height><format>R8G8B8</format></image>
+          <clip><near>0.3</near><far>100</far></clip>
+        </camera>
+      </sensor>
+      <xacro:if value="$(arg enable_training_gt)">
+        <sensor name="g2_verification_semantic_gt" type="segmentation">
+          <topic>g2/verification_semantic_gt</topic><gz_frame_id>verification_camera_depth_link</gz_frame_id>
+          <update_rate>15</update_rate><always_on>true</always_on>
+          <camera><segmentation_type>semantic</segmentation_type><optical_frame_id>verification_camera_depth_link</optical_frame_id><horizontal_fov>1.50098</horizontal_fov><image><width>640</width><height>480</height><format>R8G8B8</format></image><clip><near>0.3</near><far>100</far></clip></camera>
+        </sensor>
+        <sensor name="g2_verification_instance_gt" type="segmentation">
+          <topic>g2/verification_instance_gt</topic><gz_frame_id>verification_camera_depth_link</gz_frame_id>
+          <update_rate>15</update_rate><always_on>true</always_on>
+          <camera><segmentation_type>instance</segmentation_type><optical_frame_id>verification_camera_depth_link</optical_frame_id><horizontal_fov>1.50098</horizontal_fov><image><width>640</width><height>480</height><format>R8G8B8</format></image><clip><near>0.3</near><far>100</far></clip></camera>
+        </sensor>
+      </xacro:if>
+    </gazebo>
+  </xacro:if>
   <xacro:diff_drive_controller
     wheel_separation="${drive_wheel_separation}"
@@ -255,4 +319,11 @@
     </plugin>
   </gazebo>
+  <xacro:if value="$(arg enable_self_mask_gt)">
+    <gazebo>
+      <plugin filename="gz-sim-label-system" name="gz::sim::systems::Label">
+        <label>250</label>
+      </plugin>
+    </gazebo>
+  </xacro:if>
   <!-- 40 L bin: 0.50 * 0.40 * 0.20 = 0.040 m^3. -->
   <link name="dust_bin_link">
