Commit message: feat: add AUTO-12 efficiency design and simulator

File: starter_ws/src/sanitation_vehicle_description/urdf/sanitation_vehicle.urdf.xacro (robot description, xacro)
@@ -17,4 +17,8 @@
   <xacro:arg name="lidar_samples" default="360"/>
   <xacro:arg name="lidar_update_rate" default="10"/>
+  <!-- AUTO-12 opt-in efficiency envelope. Defaults preserve the frozen
+       0.65 m production vehicle; launch with 1.32 / 0.52 for the candidate. -->
+  <xacro:arg name="cleaning_width" default="0.65"/>
+  <xacro:arg name="brush_center_y" default="0.23"/>
   <!-- Offline G2 capture only. Production launch never overrides this false default. -->
   <xacro:arg name="enable_training_gt" default="false"/>
@@ -51,5 +55,6 @@
   <xacro:property name="wheel_pos_z" value="-0.02"/>
   <xacro:property name="wheel_mass" value="3.0"/>
-  <xacro:property name="cleaning_width" value="0.65"/>
+  <xacro:property name="cleaning_width" value="$(arg cleaning_width)"/>
+  <xacro:property name="brush_center_y" value="$(arg brush_center_y)"/>
   <xacro:property name="lidar_samples" value="$(arg lidar_samples)"/>
   <xacro:property name="lidar_update_rate" value="$(arg lidar_update_rate)"/>
@@ -348,6 +353,7 @@
     <origin xyz="-0.18 0 0.25" rpy="0 0 0"/>
   </joint>
-  <!-- Side brushes are fixed visual/collision placeholders in Stage 2.
-       Codex should add controllable joints/cleaning semantics later. -->
+  <!-- Side-brush links carry both visual and collision geometry. AUTO-12 can
+       materialize the deployed envelope by setting brush_center_y=0.52 while
+       the production default remains retracted at 0.23. -->
   <link name="left_brush_link">
     <visual>
@@ -364,5 +370,5 @@
     <parent link="base_link"/>
     <child link="left_brush_link"/>
-    <origin xyz="0.58 0.23 -0.14" rpy="0 0 0"/>
+    <origin xyz="0.58 ${brush_center_y} -0.14" rpy="0 0 0"/>
   </joint>
   <link name="right_brush_link">
@@ -380,5 +386,5 @@
     <parent link="base_link"/>
     <child link="right_brush_link"/>
-    <origin xyz="0.58 -0.23 -0.14" rpy="0 0 0"/>
+    <origin xyz="0.58 ${-brush_center_y} -0.14" rpy="0 0 0"/>
   </joint>
   <!-- Non-colliding visualization of the nominal cleaning footprint. -->

Commit message: feat(gazebo): build human-readable digital twin scene

File: starter_ws/src/sanitation_vehicle_description/urdf/sanitation_vehicle.urdf.xacro (robot description, xacro)
@@ -65,5 +65,5 @@
   <link name="base_footprint"/>
   <link name="base_link">
-    <visual>
+    <visual name="lower_chassis_visual">
       <geometry><box size="${base_length} ${base_width} ${base_height}"/></geometry>
       <material name="sanitation_chassis_yellow">
@@ -71,6 +71,48 @@
       </material>
     </visual>
-    <collision>
+    <!-- The upper body stays inside the frozen 2-D chassis envelope. Its
+         dedicated collision preserves honest vertical geometry without
+         changing navigation footprint, wheel placement, or dynamics. -->
+    <visual name="upper_body_visual">
+      <origin xyz="0.10 0 0.20" rpy="0 0 0"/>
+      <geometry><box size="0.72 0.64 0.22"/></geometry>
+      <material name="sanitation_body_white">
+        <color rgba="0.90 0.92 0.91 1.0"/>
+      </material>
+    </visual>
+    <visual name="front_service_panel_visual">
+      <origin xyz="0.49 0 0.12" rpy="0 0 0"/>
+      <geometry><box size="0.08 0.58 0.18"/></geometry>
+      <material name="sanitation_service_green">
+        <color rgba="0.02 0.43 0.27 1.0"/>
+      </material>
+    </visual>
+    <visual name="front_bumper_visual">
+      <origin xyz="0.57 0 -0.09" rpy="0 0 0"/>
+      <geometry><box size="0.06 0.74 0.08"/></geometry>
+      <material name="sanitation_bumper_dark">
+        <color rgba="0.06 0.08 0.09 1.0"/>
+      </material>
+    </visual>
+    <visual name="left_marker_visual">
+      <origin xyz="0.582 0.25 0.02" rpy="0 0 0"/>
+      <geometry><box size="0.012 0.11 0.055"/></geometry>
+      <material name="sanitation_marker_amber">
+        <color rgba="1.0 0.48 0.03 1.0"/>
+      </material>
+    </visual>
+    <visual name="right_marker_visual">
+      <origin xyz="0.582 -0.25 0.02" rpy="0 0 0"/>
+      <geometry><box size="0.012 0.11 0.055"/></geometry>
+      <material name="sanitation_marker_amber_right">
+        <color rgba="1.0 0.48 0.03 1.0"/>
+      </material>
+    </visual>
+    <collision name="lower_chassis_collision">
       <geometry><box size="${base_length} ${base_width} ${base_height}"/></geometry>
+    </collision>
+    <collision name="upper_body_collision">
+      <origin xyz="0.10 0 0.20" rpy="0 0 0"/>
+      <geometry><box size="0.72 0.64 0.22"/></geometry>
     </collision>
     <inertial>
@@ -91,8 +133,15 @@
   <xacro:macro name="sanitation_wheel" params="side pos_x pos_y red green blue">
     <link name="${side}_wheel_link">
-      <visual>
+      <visual name="tire_visual">
         <origin rpy="${pi / 2.0} 0 0"/>
         <geometry><cylinder radius="${physical_wheel_radius}" length="${wheel_width}"/></geometry>
         <material name="${side}_wheel_material">
+          <color rgba="0.035 0.045 0.05 1.0"/>
+        </material>
+      </visual>
+      <visual name="hub_visual">
+        <origin rpy="${pi / 2.0} 0 0"/>
+        <geometry><cylinder radius="${physical_wheel_radius * 0.43}" length="${wheel_width + 0.006}"/></geometry>
+        <material name="${side}_hub_material">
           <color rgba="${red} ${green} ${blue} 1.0"/>
         </material>
@@ -133,7 +182,17 @@
   <xacro:imu/>
   <link name="laser">
-    <visual>
+    <visual name="lidar_body_visual">
       <geometry><cylinder radius="0.045" length="0.06"/></geometry>
       <material name="sanitation_lidar_green"><color rgba="0.02 0.55 0.20 1.0"/></material>
+    </visual>
+    <visual name="lidar_cap_visual">
+      <origin xyz="0 0 0.031" rpy="0 0 0"/>
+      <geometry><cylinder radius="0.037" length="0.012"/></geometry>
+      <material name="sanitation_lidar_cap"><color rgba="0.03 0.04 0.05 1.0"/></material>
+    </visual>
+    <visual name="lidar_mast_visual">
+      <origin xyz="0 0 -0.115" rpy="0 0 0"/>
+      <geometry><cylinder radius="0.018" length="0.17"/></geometry>
+      <material name="sanitation_lidar_mast"><color rgba="0.20 0.23 0.24 1.0"/></material>
     </visual>
     <collision><geometry><cylinder radius="0.045" length="0.06"/></geometry></collision>
@@ -174,7 +233,12 @@
   </gazebo>
   <link name="camera_link">
-    <visual>
+    <visual name="camera_housing_visual">
       <geometry><box size="0.05 0.14 0.05"/></geometry>
-      <material name="sanitation_camera_red"><color rgba="0.45 0.05 0.05 1.0"/></material>
+      <material name="sanitation_camera_housing"><color rgba="0.08 0.10 0.11 1.0"/></material>
+    </visual>
+    <visual name="camera_lens_visual">
+      <origin xyz="0.028 0 0" rpy="0 ${pi / 2.0} 0"/>
+      <geometry><cylinder radius="0.021" length="0.012"/></geometry>
+      <material name="sanitation_camera_lens"><color rgba="0.03 0.18 0.30 1.0"/></material>
     </visual>
     <collision><geometry><box size="0.05 0.14 0.05"/></geometry></collision>
@@ -336,8 +400,18 @@
   <!-- 40 L bin: 0.50 * 0.40 * 0.20 = 0.040 m^3. -->
   <link name="dust_bin_link">
-    <visual>
+    <visual name="dust_bin_body_visual">
       <origin xyz="0 0 0"/>
       <geometry><box size="0.50 0.40 0.20"/></geometry>
       <material name="bin_green"><color rgba="0.12 0.42 0.22 1.0"/></material>
+    </visual>
+    <visual name="dust_bin_lid_visual">
+      <origin xyz="0 0 0.112"/>
+      <geometry><box size="0.52 0.42 0.025"/></geometry>
+      <material name="bin_lid_dark"><color rgba="0.04 0.12 0.09 1.0"/></material>
+    </visual>
+    <visual name="dust_bin_status_strip_visual">
+      <origin xyz="-0.251 0 0.025"/>
+      <geometry><box size="0.012 0.28 0.055"/></geometry>
+      <material name="bin_status_strip"><color rgba="0.15 0.78 0.54 1.0"/></material>
     </visual>
     <collision>
@@ -359,7 +433,17 @@
        the production default remains retracted at 0.23. -->
   <link name="left_brush_link">
-    <visual>
+    <visual name="left_brush_hub_visual">
       <geometry><cylinder radius="0.14" length="0.03"/></geometry>
       <material name="left_brush_dark"><color rgba="0.08 0.08 0.08 1.0"/></material>
+    </visual>
+    <visual name="left_brush_cross_visual">
+      <origin xyz="0 0 -0.018"/>
+      <geometry><box size="0.30 0.035 0.012"/></geometry>
+      <material name="left_brush_bristle"><color rgba="0.38 0.24 0.08 1.0"/></material>
+    </visual>
+    <visual name="left_brush_cross_visual_2">
+      <origin xyz="0 0 -0.018" rpy="0 0 ${pi / 2.0}"/>
+      <geometry><box size="0.30 0.035 0.012"/></geometry>
+      <material name="left_brush_bristle_2"><color rgba="0.38 0.24 0.08 1.0"/></material>
     </visual>
     <collision><geometry><cylinder radius="0.14" length="0.03"/></geometry></collision>
@@ -375,7 +459,17 @@
   </joint>
   <link name="right_brush_link">
-    <visual>
+    <visual name="right_brush_hub_visual">
       <geometry><cylinder radius="0.14" length="0.03"/></geometry>
       <material name="right_brush_dark"><color rgba="0.09 0.09 0.09 1.0"/></material>
+    </visual>
+    <visual name="right_brush_cross_visual">
+      <origin xyz="0 0 -0.018"/>
+      <geometry><box size="0.30 0.035 0.012"/></geometry>
+      <material name="right_brush_bristle"><color rgba="0.38 0.24 0.08 1.0"/></material>
+    </visual>
+    <visual name="right_brush_cross_visual_2">
+      <origin xyz="0 0 -0.018" rpy="0 0 ${pi / 2.0}"/>
+      <geometry><box size="0.30 0.035 0.012"/></geometry>
+      <material name="right_brush_bristle_2"><color rgba="0.38 0.24 0.08 1.0"/></material>
     </visual>
     <collision><geometry><cylinder radius="0.14" length="0.03"/></geometry></collision>

Commit message: feat: add native Gazebo cleaning controls and scene scales

File: starter_ws/src/sanitation_vehicle_description/urdf/sanitation_vehicle.urdf.xacro (robot description, xacro)
@@ -108,4 +108,69 @@
         <color rgba="1.0 0.48 0.03 1.0"/>
       </material>
+    </visual>
+    <visual name="left_headlamp_visual">
+      <origin xyz="0.585 0.18 0.11" rpy="0 0 0"/>
+      <geometry><box size="0.014 0.13 0.075"/></geometry>
+      <material name="headlamp_white"><color rgba="0.92 0.96 1.0 1.0"/></material>
+    </visual>
+    <visual name="right_headlamp_visual">
+      <origin xyz="0.585 -0.18 0.11" rpy="0 0 0"/>
+      <geometry><box size="0.014 0.13 0.075"/></geometry>
+      <material name="headlamp_white_right"><color rgba="0.92 0.96 1.0 1.0"/></material>
+    </visual>
+    <visual name="left_rear_lamp_visual">
+      <origin xyz="-0.585 0.25 0.05" rpy="0 0 0"/>
+      <geometry><box size="0.014 0.12 0.07"/></geometry>
+      <material name="rear_lamp_red"><color rgba="0.82 0.03 0.025 1.0"/></material>
+    </visual>
+    <visual name="right_rear_lamp_visual">
+      <origin xyz="-0.585 -0.25 0.05" rpy="0 0 0"/>
+      <geometry><box size="0.014 0.12 0.07"/></geometry>
+      <material name="rear_lamp_red_right"><color rgba="0.82 0.03 0.025 1.0"/></material>
+    </visual>
+    <visual name="left_access_door_visual">
+      <origin xyz="0.10 0.326 0.20" rpy="0 0 0"/>
+      <geometry><box size="0.48 0.012 0.16"/></geometry>
+      <material name="access_door_gray"><color rgba="0.70 0.74 0.75 1.0"/></material>
+    </visual>
+    <visual name="right_access_door_visual">
+      <origin xyz="0.10 -0.326 0.20" rpy="0 0 0"/>
+      <geometry><box size="0.48 0.012 0.16"/></geometry>
+      <material name="access_door_gray_right"><color rgba="0.70 0.74 0.75 1.0"/></material>
+    </visual>
+    <visual name="left_door_handle_visual">
+      <origin xyz="0.28 0.334 0.23" rpy="0 0 0"/>
+      <geometry><box size="0.10 0.016 0.025"/></geometry>
+      <material name="door_handle_dark"><color rgba="0.05 0.07 0.08 1.0"/></material>
+    </visual>
+    <visual name="right_door_handle_visual">
+      <origin xyz="0.28 -0.334 0.23" rpy="0 0 0"/>
+      <geometry><box size="0.10 0.016 0.025"/></geometry>
+      <material name="door_handle_dark_right"><color rgba="0.05 0.07 0.08 1.0"/></material>
+    </visual>
+    <visual name="charging_port_visual">
+      <origin xyz="-0.22 -0.337 0.20" rpy="${pi / 2.0} 0 0"/>
+      <geometry><cylinder radius="0.055" length="0.018"/></geometry>
+      <material name="charging_port_blue"><color rgba="0.04 0.28 0.52 1.0"/></material>
+    </visual>
+    <visual name="roof_safety_beacon_visual">
+      <origin xyz="-0.10 0 0.36" rpy="0 0 0"/>
+      <geometry><cylinder radius="0.07" length="0.11"/></geometry>
+      <material name="safety_beacon_amber"><color rgba="1.0 0.38 0.01 0.95"/></material>
+    </visual>
+    <visual name="rear_suction_intake_visual">
+      <origin xyz="-0.50 0 -0.13" rpy="0 0 0"/>
+      <geometry><box size="0.18 0.54 0.055"/></geometry>
+      <material name="suction_intake_dark"><color rgba="0.035 0.05 0.055 1.0"/></material>
+    </visual>
+    <visual name="left_safety_stripe_visual">
+      <origin xyz="-0.23 0.337 0.08" rpy="0 0 0"/>
+      <geometry><box size="0.32 0.010 0.055"/></geometry>
+      <material name="safety_stripe_green"><color rgba="0.02 0.52 0.30 1.0"/></material>
+    </visual>
+    <visual name="right_safety_stripe_visual">
+      <origin xyz="-0.23 -0.337 0.08" rpy="0 0 0"/>
+      <geometry><box size="0.32 0.010 0.055"/></geometry>
+      <material name="safety_stripe_green_right"><color rgba="0.02 0.52 0.30 1.0"/></material>
     </visual>
     <collision name="lower_chassis_collision">
@@ -433,4 +498,9 @@
        the production default remains retracted at 0.23. -->
   <link name="left_brush_link">
+    <visual name="left_brush_support_arm_visual">
+      <origin xyz="-0.12 -0.06 0.025" rpy="0 0 -0.35"/>
+      <geometry><box size="0.30 0.045 0.045"/></geometry>
+      <material name="left_brush_support_green"><color rgba="0.02 0.43 0.27 1.0"/></material>
+    </visual>
     <visual name="left_brush_hub_visual">
       <geometry><cylinder radius="0.14" length="0.03"/></geometry>
@@ -459,4 +529,9 @@
   </joint>
   <link name="right_brush_link">
+    <visual name="right_brush_support_arm_visual">
+      <origin xyz="-0.12 0.06 0.025" rpy="0 0 0.35"/>
+      <geometry><box size="0.30 0.045 0.045"/></geometry>
+      <material name="right_brush_support_green"><color rgba="0.02 0.43 0.27 1.0"/></material>
+    </visual>
     <visual name="right_brush_hub_visual">
       <geometry><cylinder radius="0.14" length="0.03"/></geometry>
