Commit message: feat(vehicle): add integrated functional acceptance

File: starter_ws/src/sanitation_vehicle_description/urdf/formal_competition_vehicle.urdf.xacro (robot description, xacro)
@@ -38,4 +38,19 @@
         <wastewater_capacity_kg>9.7064</wastewater_capacity_kg>
       </plugin>
+      <plugin filename="libWaterRecoverySystem.so" name="sanitation_gazebo_control::WaterRecoverySystem">
+        <pump_rated_flow_l_min>15.1</pump_rated_flow_l_min>
+        <hydraulic_derating>0.70</hydraulic_derating>
+        <tank_capacity_kg>9.7064</tank_capacity_kg>
+        <initial_tank_mass_kg>0.0</initial_tank_mass_kg>
+        <initial_ground_volume_l>2.88</initial_ground_volume_l>
+        <water_density_kg_l>1.0</water_density_kg_l>
+        <patch_min_x>-0.60</patch_min_x><patch_max_x>1.80</patch_max_x>
+        <patch_min_y>-0.30</patch_min_y><patch_max_y>0.30</patch_max_y>
+        <cell_size_m>0.10</cell_size_m>
+        <nozzle_length_m>0.14</nozzle_length_m>
+        <nozzle_width_m>0.65</nozzle_width_m>
+        <maximum_squeegee_clearance_m>0.012</maximum_squeegee_clearance_m>
+        <maximum_intake_clearance_m>0.012</maximum_intake_clearance_m>
+      </plugin>
     </gazebo>
   </xacro:if>

File: starter_ws/src/sanitation_vehicle_description/urdf/high_fidelity/bodywork.xacro (robot description, xacro)
@@ -94,7 +94,12 @@
       <xacro:hf_body_visual mesh="arm_bay_rear_sill.stl" material="arm_bay_sill" rgba="0.075 0.090 0.092 1" visible="${visible}"/>
       <collision name="nose_collision"><origin xyz="0.32 0 0.280"/><geometry><box size="0.47 0.65 0.20"/></geometry></collision>
-      <collision name="power_cowl_collision"><origin xyz="0.28 0.235 0.535"/><geometry><box size="0.49 0.29 0.48"/></geometry></collision>
+      <!-- Keep the aft face ahead of the dry-bin front panel.  The former
+           490 mm box entered the certified dry usable envelope by 2.5 mm. -->
+      <collision name="power_cowl_collision"><origin xyz="0.290 0.235 0.535"/><geometry><box size="0.470 0.29 0.48"/></geometry></collision>
       <collision name="compute_cowl_collision"><origin xyz="0.31 -0.285 0.365"/><geometry><box size="0.39 0.19 0.22"/></geometry></collision>
-      <collision name="arm_bay_floor_collision"><origin xyz="0.17 -0.20 0.33"/><geometry><box size="0.58 0.40 0.10"/></geometry></collision>
+      <!-- The arm bay is a forward body tray; the payload deck and dedicated
+           arm adapter carry the manipulator.  Its collision therefore ends at
+           x=0.055 m and cannot become a hidden shelf through either tank. -->
+      <collision name="arm_bay_floor_collision"><origin xyz="0.2575 -0.20 0.33"/><geometry><box size="0.405 0.40 0.10"/></geometry></collision>
       <xacro:hf_bodywork_box_inertial mass="3.40" sx="0.58" sy="0.72" sz="0.55" xyz="0.26 0.06 0.43"/>
     </link>
@@ -111,7 +116,17 @@
            make a visually open hopper physically unusable. -->
       <collision name="rear_shell_rear_wall_collision"><origin xyz="-0.540 0 0.495"/><geometry><box size="0.045 0.70 0.52"/></geometry></collision>
-      <collision name="rear_shell_left_wall_collision"><origin xyz="-0.285 0.365 0.495"/><geometry><box size="0.53 0.045 0.52"/></geometry></collision>
-      <collision name="rear_shell_right_wall_collision"><origin xyz="-0.285 -0.365 0.495"/><geometry><box size="0.53 0.045 0.52"/></geometry></collision>
-      <collision name="rear_shell_lower_collision"><origin xyz="-0.285 0 0.350"/><geometry><box size="0.53 0.68 0.23"/></geometry></collision>
+      <!-- Thin moulded outer panels sit beyond the independent tank boards.
+           Their inner faces retain 3.5 mm (dry) and 4 mm (wet) installation
+           gaps instead of duplicating the internal walls with overlapping
+           45 mm collision solids. -->
+      <collision name="rear_shell_left_wall_collision"><origin xyz="-0.285 0.365 0.495"/><geometry><box size="0.53 0.020 0.52"/></geometry></collision>
+      <collision name="rear_shell_right_wall_collision"><origin xyz="-0.285 -0.388 0.495"/><geometry><box size="0.53 0.020 0.52"/></geometry></collision>
+      <!-- The moulded lower return is a perimeter frame, not a solid shelf.
+           Keep its three load-bearing outer rails outside the dry / wet tank
+           clear volumes so the robot chute remains a continuous gravity path
+           to the real dry-bin floor. -->
+      <collision name="rear_shell_lower_left_skirt_collision"><origin xyz="-0.285 0.365 0.275"/><geometry><box size="0.53 0.020 0.080"/></geometry></collision>
+      <collision name="rear_shell_lower_right_skirt_collision"><origin xyz="-0.285 -0.388 0.275"/><geometry><box size="0.53 0.020 0.080"/></geometry></collision>
+      <collision name="rear_shell_lower_rear_rail_collision"><origin xyz="-0.540 0 0.275"/><geometry><box size="0.045 0.70 0.080"/></geometry></collision>
       <collision name="rear_shell_roof_left_collision"><origin xyz="-0.285 0.310 0.735"/><geometry><box size="0.53 0.080 0.055"/></geometry></collision>
       <collision name="rear_shell_roof_right_collision"><origin xyz="-0.285 -0.255 0.735"/><geometry><box size="0.53 0.180 0.055"/></geometry></collision>

File: starter_ws/src/sanitation_vehicle_description/urdf/high_fidelity/cleaning_mechanism.xacro (robot description, xacro)
@@ -279,5 +279,8 @@
     <joint name="squeegee_float_joint" type="prismatic">
       <parent link="cleaning_lift_carriage_link"/><child link="squeegee_float_carrier_link"/>
-      <origin xyz="-0.445 0 -0.011" rpy="0 0 0"/>
+      <!-- The carrier datum puts the rubber blade on the ground plane at the
+           nominal lowered lift position; the prismatic axis then supplies its
+           measured +/-15 mm compliance instead of leaving the blade floating. -->
+      <origin xyz="-0.445 0 -0.051" rpy="0 0 0"/>
       <axis xyz="0 0 1"/>
       <limit lower="-0.015" upper="0.015" effort="250.0" velocity="0.10"/>
@@ -320,5 +323,7 @@
     <joint name="suction_nozzle_mount_joint" type="fixed">
       <parent link="squeegee_link"/><child link="suction_nozzle_link"/>
-      <origin xyz="0.040 0 0.010" rpy="0 0 0"/>
+      <!-- The intake box bottom retains a nominal 4-6 mm gap while the rubber
+           squeegee blade is grounded; the intake itself must not scrape. -->
+      <origin xyz="0.040 0 -0.005" rpy="0 0 0"/>
     </joint>
     <gazebo reference="suction_nozzle_link">

File: starter_ws/src/sanitation_vehicle_description/urdf/high_fidelity/storage_system.xacro (robot description, xacro)
@@ -157,5 +157,19 @@
       <xacro:hf_storage_visual mesh="dry_deposit_chute.stl"
         material="hf_deposit_chute" rgba="0.20 0.48 0.32 1"/>
-      <collision name="dry_deposit_chute_collision"><geometry><box size="0.125 0.100 0.350"/></geometry></collision>
+      <!-- The chute is a gravity passage, not a solid block.  Four thin wall
+           collisions retain a 109 x 84 mm clear bore for the 30 mm cube and
+           leave both ends open. -->
+      <collision name="dry_deposit_chute_front_wall_collision">
+        <origin xyz="0.0585 0 0"/><geometry><box size="0.008 0.100 0.350"/></geometry>
+      </collision>
+      <collision name="dry_deposit_chute_rear_wall_collision">
+        <origin xyz="-0.0585 0 0"/><geometry><box size="0.008 0.100 0.350"/></geometry>
+      </collision>
+      <collision name="dry_deposit_chute_left_wall_collision">
+        <origin xyz="0 0.046 0"/><geometry><box size="0.109 0.008 0.350"/></geometry>
+      </collision>
+      <collision name="dry_deposit_chute_right_wall_collision">
+        <origin xyz="0 -0.046 0"/><geometry><box size="0.109 0.008 0.350"/></geometry>
+      </collision>
       <xacro:hf_storage_box_inertial mass="0.320" sx="0.130" sy="0.105" sz="0.350"/>
     </link>
@@ -177,5 +191,8 @@
       <sensor name="dry_deposit_contact" type="contact">
         <topic>/storage/dry_deposit/contact</topic><update_rate>50</update_rate><always_on>true</always_on>
-        <contact><collision>dry_deposit_chute_collision</collision></contact>
+        <!-- Fixed-joint reduction merges the chute into the actuated lid and
+             prefixes the final SDF collision.  Reference that physics name so
+             the acceptance contact topic contains real samples. -->
+        <contact><collision>dry_bin_lid_link_fixed_joint_lump__dry_deposit_chute_front_wall_collision_collision_8</collision></contact>
       </sensor>
     </gazebo>

Commit message: fix(vehicle): harden formal model provenance

File: starter_ws/src/sanitation_vehicle_description/urdf/formal_competition_vehicle.urdf.xacro (robot description, xacro)
@@ -45,4 +45,6 @@
         <dry_capacity_kg>1.512</dry_capacity_kg>
         <wastewater_capacity_kg>9.7064</wastewater_capacity_kg>
+        <initial_dry_mass_kg>$(arg dry_load_mass_kg)</initial_dry_mass_kg>
+        <initial_wastewater_mass_kg>$(arg wastewater_load_mass_kg)</initial_wastewater_mass_kg>
       </plugin>
       <plugin filename="libWaterRecoverySystem.so" name="sanitation_gazebo_control::WaterRecoverySystem">
@@ -50,5 +52,5 @@
         <hydraulic_derating>0.70</hydraulic_derating>
         <tank_capacity_kg>9.7064</tank_capacity_kg>
-        <initial_tank_mass_kg>0.0</initial_tank_mass_kg>
+        <initial_tank_mass_kg>$(arg wastewater_load_mass_kg)</initial_tank_mass_kg>
         <initial_ground_volume_l>2.88</initial_ground_volume_l>
         <water_density_kg_l>1.0</water_density_kg_l>

File: starter_ws/src/sanitation_vehicle_description/urdf/high_fidelity/storage_system.xacro (robot description, xacro)
@@ -70,8 +70,8 @@
     <xacro:property name="wet_center_y" value="-0.245"/>
     <xacro:property name="panel_t" value="0.004"/>
-    <xacro:property name="dry_payload_mass" value="${max(float(dry_load_mass_kg), 0.001)}"/>
-    <xacro:property name="water_payload_mass" value="${max(float(wastewater_load_mass_kg), 0.001)}"/>
+    <xacro:property name="dry_payload_mass" value="${max(min(float(dry_load_mass_kg), 1.512), 0.001)}"/>
+    <xacro:property name="water_payload_mass" value="${max(min(float(wastewater_load_mass_kg), 9.7064), 0.001)}"/>
     <xacro:property name="water_fill_height"
-                    value="${min(water_payload_mass / (1000.0 * wet_inner_x * wet_inner_y), 0.009706 / (wet_inner_x * wet_inner_y))}"/>
+                    value="${water_payload_mass / (1000.0 * wet_inner_x * wet_inner_y)}"/>
     <link name="storage_system_mount_link">
       <xacro:hf_storage_visual mesh="storage_mount_tray.stl"

Commit message: feat: harden public DOSOD evidence pipeline

File: starter_ws/src/sanitation_vehicle_description/urdf/formal_competition_vehicle.urdf.xacro (robot description, xacro)
@@ -20,4 +20,5 @@
   <xacro:arg name="bodywork_visible" default="true"/>
   <xacro:arg name="high_bandwidth_sensor_runtime" default="true"/>
+  <xacro:arg name="enable_training_gt" default="false"/>
   <xacro:arg name="service_acceptance_interfaces" default="false"/>
   <xacro:arg name="service_door_evaluation_interfaces" default="false"/>
@@ -40,5 +41,6 @@
   <xacro:hf_manipulator_stack parent="arm_mount_link" use_sim="$(arg use_sim)"/>
   <xacro:hf_sensor_suite mast_parent="sensor_mast_link" base_parent="base_link" wrist_parent="tool0"
-                         high_bandwidth_runtime="$(arg high_bandwidth_sensor_runtime)"/>
+                         high_bandwidth_runtime="$(arg high_bandwidth_sensor_runtime)"
+                         enable_training_gt="$(arg enable_training_gt)"/>
   <xacro:high_fidelity_cleaning_mechanism parent="base_link" origin_xyz="0 0 0" origin_rpy="0 0 0"/>
   <xacro:high_fidelity_storage_system

File: starter_ws/src/sanitation_vehicle_description/urdf/high_fidelity/sensor_suite.xacro (robot description, xacro)
@@ -20,5 +20,5 @@
     </joint>
   </xacro:macro>
-  <xacro:macro name="hf_d435" params="name parent xyz rpy topic ir_left_topic ir_right_topic max_range mount_bracket:=false runtime_enabled:=true">
+  <xacro:macro name="hf_d435" params="name parent xyz rpy topic ir_left_topic ir_right_topic max_range mount_bracket:=false runtime_enabled:=true training_gt:=false">
     <xacro:if value="${mount_bracket}">
       <link name="${name}_mount_link">
@@ -107,4 +107,15 @@
         </camera>
       </sensor>
+      <xacro:if value="${training_gt}">
+        <!-- Evidence-only labels share the production D435 link, lens and cadence. -->
+        <sensor name="g2_semantic_gt" type="segmentation">
+          <topic>g2/semantic_gt</topic><gz_frame_id>${name}_depth_optical_frame</gz_frame_id><update_rate>30</update_rate><always_on>true</always_on>
+          <camera><segmentation_type>semantic</segmentation_type><optical_frame_id>${name}_depth_optical_frame</optical_frame_id><horizontal_fov>1.518436</horizontal_fov><image><width>848</width><height>480</height><format>R8G8B8</format></image><clip><near>0.2</near><far>${max_range}</far></clip><lens><intrinsics><fx>447.2</fx><fy>433.0</fy><cx>424.0</cx><cy>240.0</cy><s>0</s></intrinsics></lens></camera>
+        </sensor>
+        <sensor name="g2_instance_gt" type="segmentation">
+          <topic>g2/instance_gt</topic><gz_frame_id>${name}_depth_optical_frame</gz_frame_id><update_rate>30</update_rate><always_on>true</always_on>
+          <camera><segmentation_type>instance</segmentation_type><optical_frame_id>${name}_depth_optical_frame</optical_frame_id><horizontal_fov>1.518436</horizontal_fov><image><width>848</width><height>480</height><format>R8G8B8</format></image><clip><near>0.2</near><far>${max_range}</far></clip><lens><intrinsics><fx>447.2</fx><fy>433.0</fy><cx>424.0</cx><cy>240.0</cy><s>0</s></intrinsics></lens></camera>
+        </sensor>
+      </xacro:if>
       <sensor name="${name}_d435_infra1" type="camera">
         <pose>0 0 0 0 0 0</pose>
@@ -184,5 +195,5 @@
     </xacro:if>
   </xacro:macro>
-  <xacro:macro name="hf_sensor_suite" params="mast_parent base_parent wrist_parent high_bandwidth_runtime:=true">
+  <xacro:macro name="hf_sensor_suite" params="mast_parent base_parent wrist_parent high_bandwidth_runtime:=true enable_training_gt:=false">
     <!-- Every fixed sensor is connected through a named, physical mounting
          link.  This makes the installation hierarchy inspectable in TF/URDF
@@ -275,5 +286,5 @@
                     ir_left_topic="/sensors/front_rgbd/infra1/image_rect_raw"
                     ir_right_topic="/sensors/front_rgbd/infra2/image_rect_raw" max_range="10.0"
-                    runtime_enabled="${high_bandwidth_runtime}"/>
+                    runtime_enabled="${high_bandwidth_runtime}" training_gt="${enable_training_gt}"/>
     <!-- Side bracket position keeps the camera outside the Robotiq base and
          turns its optical +X onto the gripper's +Z approach direction. -->
