Commit message: Model self-locking cleaning lift hold

File: starter_ws/src/sanitation_vehicle_description/urdf/high_fidelity/cleaning_mechanism.xacro (robot description, xacro)
@@ -229,5 +229,9 @@
            4.8 mm/s no-load speed from the public manufacturer sheet. -->
       <limit lower="0.0" upper="0.100" effort="300.0" velocity="0.0048"/>
-      <dynamics damping="80.0" friction="35.0"/>
+      <!-- The moving cleaning subtree is 5.95 kg (58.35 N under gravity).
+           Model the P16 screw actuator's non-backdrivable hold with 80 N of
+           static resistance: above the suspended load, but well below the
+           actuator's 300 N commanded-force envelope. -->
+      <dynamics damping="80.0" friction="80.0"/>
     </joint>
     <!-- Actuonix P16 body is chassis-fixed; its rod and clevis ride with the carriage. -->

Commit message: Harden formal function-position runtime evidence

File: starter_ws/src/sanitation_vehicle_description/urdf/high_fidelity/cleaning_mechanism.xacro (robot description, xacro)
@@ -459,5 +459,8 @@
         <update_rate>100</update_rate>
         <always_on>true</always_on>
-        <contact><collision>squeegee_blade_collision</collision></contact>
+        <!-- sdformat folds the fixed suction-nozzle child into squeegee_link and
+             consequently renames this URDF collision in the generated SDF.
+             Contact sensors bind against that post-conversion SDF name. -->
+        <contact><collision>squeegee_link_fixed_joint_lump__squeegee_blade_collision_collision</collision></contact>
       </sensor>
     </gazebo>

File: starter_ws/src/sanitation_vehicle_description/urdf/high_fidelity/control_interfaces.xacro (robot description, xacro)
@@ -89,5 +89,8 @@
            charge lock, E-stop plunger and service lids are passive joints and
            intentionally have no ros2_control command interface. -->
-      <xacro:hf_position_joint name="wastewater_drain_valve_joint" lower="0.0" upper="${pi/2.0}" velocity="1.2" effort="25.0"/>
+      <!-- Keep the powered valve just 20 microradians off the exact DART
+           lower stop.  This is far below the closed-state threshold while
+           avoiding a locked unilateral constraint on the opening command. -->
+      <xacro:hf_position_joint name="wastewater_drain_valve_joint" lower="0.0" upper="${pi/2.0}" velocity="1.2" effort="25.0" initial_position="0.00002"/>
       <!-- Passive service hardware is not commandable, but its measured
            position must reach joint_state_broadcaster for physical interlocks. -->

Commit message: Allow lift retraction from physical travel stop

File: starter_ws/src/sanitation_vehicle_description/urdf/high_fidelity/cleaning_mechanism.xacro (robot description, xacro)
@@ -230,8 +230,10 @@
       <limit lower="0.0" upper="0.100" effort="300.0" velocity="0.0048"/>
       <!-- The moving cleaning subtree is 5.95 kg (58.35 N under gravity).
-           Model the P16 screw actuator's non-backdrivable hold with 80 N of
-           static resistance: above the suspended load, but well below the
-           actuator's 300 N commanded-force envelope. -->
-      <dynamics damping="80.0" friction="80.0"/>
+           URDF friction is direction-symmetric, so it cannot represent the
+           P16 screw's powered/non-powered one-way hold.  Keep the calibrated
+           80 Ns/m damping and use 60 N breakaway drag: it remains above the
+           suspended load for passive hold while leaving a realistic margin for
+           powered reverse release from the 100 mm physical stop. -->
+      <dynamics damping="80.0" friction="60.0"/>
     </joint>
     <!-- Actuonix P16 body is chassis-fixed; its rod and clevis ride with the carriage. -->

Commit message: Keep lift stop reversible in DART

File: starter_ws/src/sanitation_vehicle_description/urdf/high_fidelity/cleaning_mechanism.xacro (robot description, xacro)
@@ -228,12 +228,17 @@
       <!-- Actuonix P16-100-256-12-P: 300 N maximum lifted load and
            4.8 mm/s no-load speed from the public manufacturer sheet. -->
-      <limit lower="0.0" upper="0.100" effort="300.0" velocity="0.0048"/>
+      <!-- Keep DART's solver bound 20 um beyond the product's 100 mm travel
+           contract.  The ros2_control position interface remains capped at
+           0.100 m, so product commands and all acceptance thresholds retain
+           the P16's 100 mm stroke.  This small reversible clearance prevents
+           DART from locking an outward-driven prismatic joint in its exact
+           unilateral upper-limit constraint, which would otherwise make a
+           legitimate post-fault retraction physically impossible. -->
+      <limit lower="0.0" upper="0.10002" effort="300.0" velocity="0.0048"/>
       <!-- The moving cleaning subtree is 5.95 kg (58.35 N under gravity).
-           URDF friction is direction-symmetric, so it cannot represent the
-           P16 screw's powered/non-powered one-way hold.  Keep the calibrated
-           80 Ns/m damping and use 60 N breakaway drag: it remains above the
-           suspended load for passive hold while leaving a realistic margin for
-           powered reverse release from the 100 mm physical stop. -->
-      <dynamics damping="80.0" friction="60.0"/>
+           Keep the calibrated 80 Ns/m damping and 80 N breakaway drag; URDF
+           friction is direction-symmetric and is not a substitute for the
+           P16 screw's powered/non-powered one-way holding behaviour. -->
+      <dynamics damping="80.0" friction="80.0"/>
     </joint>
     <!-- Actuonix P16 body is chassis-fixed; its rod and clevis ride with the carriage. -->
