Commit message: Close final visual preview runtime gaps

File: starter_ws/src/sanitation_vehicle_description/urdf/high_fidelity/a300_platform.xacro (robot description, xacro)
@@ -20,5 +20,5 @@
         <material name="${name}_tire"><color rgba="0.035 0.040 0.045 1"/></material>
       </visual>
-      <collision name="${name}_wheel_collision">
+      <collision>
         <origin rpy="${pi/2.0} 0 0"/>
         <geometry><cylinder radius="0.1651" length="0.1143"/></geometry>
@@ -38,6 +38,11 @@
       <dynamics damping="0.15" friction="0.05"/>
     </joint>
+    <!-- URDF-to-SDF only applies this link extension to its unnamed primary
+         collision. A named wheel collision silently lost the whole surface
+         block and left DART's isotropic 1.0 default in runtime. -->
     <gazebo reference="${name}_wheel_link">
       <mu1>0.9</mu1><mu2>0.72</mu2>
+      <!-- collision-local X is the rolling / vehicle-longitudinal direction -->
+      <fdir1>1 0 0</fdir1>
       <kp>1000000</kp><kd>100</kd>
       <minDepth>0.001</minDepth><maxVel>0.1</maxVel>

Commit message: fix: preserve A300 wheel contact surfaces in SDF conversion

File: starter_ws/src/sanitation_vehicle_description/urdf/high_fidelity/a300_platform.xacro (robot description, xacro)
@@ -21,5 +21,5 @@
         <material name="${name}_tire"><color rgba="0.035 0.040 0.045 1"/></material>
       </visual>
-      <collision name="${name}_wheel_collision">
+      <collision>
         <origin rpy="${pi/2.0} 0 0"/>
         <geometry><cylinder radius="0.1651" length="0.1143"/></geometry>
@@ -39,6 +39,11 @@
       <dynamics damping="0.15" friction="0.05"/>
     </joint>
+    <!-- URDF-to-SDF only applies this link extension to its unnamed primary
+         collision. A named wheel collision silently lost the whole surface
+         block and left DART's isotropic 1.0 default in runtime. -->
     <gazebo reference="${name}_wheel_link">
       <mu1>0.9</mu1><mu2>0.72</mu2>
+      <!-- collision-local X is the rolling / vehicle-longitudinal direction -->
+      <fdir1>1 0 0</fdir1>
       <kp>1000000</kp><kd>100</kd>
       <minDepth>0.001</minDepth><maxVel>0.1</maxVel>
