Commit message: feat: deliver product-grade formal vehicle bodywork

File: reports/engineering/formal_competition_vehicle.urdf (robot description, URDF)
Before this commit: robot tzcup_formal_sanitation_vehicle, 105 links, 104 joints
Links:
- added link bodywork_brush_guards_link, mass 0.36; collision box size=0.15 0.14 0.10; collision box size=0.15 0.14 0.10
- added link bodywork_compute_service_door_link, mass 0.16; collision box size=0.31 0.010 0.18; visual mesh filename=package://sanitation_vehicle_description/meshes/project/bod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
- added link bodywork_front_cowl_link, mass 3.4; collision box size=0.39 0.19 0.22; collision box size=0.47 0.65 0.20
- added link bodywork_lighting_link, mass 0.34; collision cylinder length=0.040 radius=0.026; visual mesh filename=package://sanitation_vehicle_description/meshes/project/bod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
- added link bodywork_lower_tub_link, mass 3.8; collision box size=0.055 0.660 0.070; collision box size=0.060 0.700 0.075
- added link bodywork_power_service_door_link, mass 0.28; collision box size=0.45 0.010 0.43; visual mesh filename=package://sanitation_vehicle_description/meshes/project/bod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
- added link bodywork_rear_dry_service_door_link, mass 0.3; collision box size=0.012 0.44 0.35; visual mesh filename=package://sanitation_vehicle_description/meshes/project/bod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
- added link bodywork_rear_shell_link, mass 3.1; collision box size=0.13 0.15 0.35; collision box size=0.53 0.70 0.52
- added link bodywork_trim_link, mass 0.42; collision cylinder length=0.020 radius=0.032; collision cylinder length=0.065 radius=0.025
- added link bodywork_wet_service_door_link, mass 0.22; collision box size=0.37 0.010 0.29; visual mesh filename=package://sanitation_vehicle_description/meshes/project/bod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
- link arm_mount_link: mass 0.001 -> 2.8
- link sensor_mast_link: geometry collision box size=0.040 0.040 0.130; collision box size=0.060 0.060 0.850
Joints:
- added joint bodywork_brush_guards_joint: type fixed, parent base_link, child bodywork_brush_guards_link
- added joint bodywork_compute_service_door_joint: type fixed, parent base_link, child bodywork_compute_service_door_link, origin xyz=0 0 0 rpy=0 0 0
- added joint bodywork_front_cowl_joint: type fixed, parent base_link, child bodywork_front_cowl_link
- added joint bodywork_lighting_joint: type fixed, parent base_link, child bodywork_lighting_link
- added joint bodywork_lower_tub_joint: type fixed, parent base_link, child bodywork_lower_tub_link
- added joint bodywork_power_service_door_joint: type fixed, parent base_link, child bodywork_power_service_door_link, origin xyz=0 0 0 rpy=0 0 0
- added joint bodywork_rear_dry_service_door_joint: type fixed, parent base_link, child bodywork_rear_dry_service_door_link, origin xyz=0 0 0 rpy=0 0 0
- added joint bodywork_rear_shell_joint: type fixed, parent base_link, child bodywork_rear_shell_link
- added joint bodywork_trim_joint: type fixed, parent base_link, child bodywork_trim_link
- added joint bodywork_wet_service_door_joint: type fixed, parent base_link, child bodywork_wet_service_door_link, origin xyz=0 0 0 rpy=0 0 0
- joint arm_mount_joint: origin xyz=0.035 -0.145 0.065 -> xyz=0.100 -0.200 0.065
- joint front_rgbd_mount_joint: origin xyz=0.640 0 0.225 rpy=0 0 0 -> xyz=0.570 0 0.449 rpy=0 0 0; parent sensor_mast_link -> base_link
- joint gnss_antenna_mount_joint: origin xyz=0 0 0.845 -> xyz=-0.100 0 0.965
- joint lidar_2d_mount_joint: origin xyz=0.380 0 0.395 -> xyz=0.250 0 0.665; parent sensor_mast_link -> base_link
- joint lidar_3d_mount_joint: origin xyz=0 0 0.725 -> xyz=0 0 0.845
- joint rear_left_fisheye_mount_joint: origin xyz=-0.350 0.275 0.200 rpy=0 -0.175 2.705 -> xyz=-0.565 0.280 0.435 rpy=0 -0.175 2.705; parent sensor_mast_link -> base_link
- joint rear_right_fisheye_mount_joint: origin xyz=-0.350 -0.275 0.200 rpy=0 -0.175 -2.705 -> xyz=-0.565 -0.280 0.435 rpy=0 -0.175 -2.705; parent sensor_mast_link -> base_link
- joint recovery_hose_lower_joint: origin xyz=-0.08 0 0.10 rpy=0 -0.58 0 -> xyz=-0.470 0 0.100 rpy=0 -0.750 0; parent suction_nozzle_link -> cleaning_mechanism_mount_link
- joint recovery_hose_middle_joint: origin xyz=-0.16 0 0.10 rpy=0 -0.70 0 -> xyz=-0.320 0 0.280 rpy=0 -0.950 0; parent recovery_hose_lower_link -> cleaning_mechanism_mount_link
- joint recovery_hose_upper_joint: origin xyz=-0.17 0 0.14 rpy=0 -0.35 0 -> xyz=-0.202 0 0.471 rpy=0 -1.100 0; parent recovery_hose_middle_link -> cleaning_mechanism_mount_link
- joint ur5e_mount_joint: origin xyz=0 0 0.015 -> xyz=0 0 0.045

File: starter_ws/src/sanitation_vehicle_description/urdf/formal_competition_vehicle.urdf.xacro (robot description, xacro)
@@ -6,8 +6,10 @@
   <xacro:include filename="high_fidelity/cleaning_mechanism.xacro"/>
   <xacro:include filename="high_fidelity/storage_system.xacro"/>
+  <xacro:include filename="high_fidelity/bodywork.xacro"/>
   <xacro:include filename="high_fidelity/control_interfaces.xacro"/>
   <xacro:arg name="use_sim" default="true"/>
   <xacro:arg name="dry_load_mass_kg" default="0.0"/>
   <xacro:arg name="wastewater_load_mass_kg" default="0.0"/>
+  <xacro:arg name="bodywork_visible" default="true"/>
   <!-- The unloaded vehicle is the default. Load-state variants are generated
        by setting the two mass arguments; runtime collection accounting must
@@ -23,4 +25,5 @@
       dry_load_mass_kg="$(arg dry_load_mass_kg)"
       wastewater_load_mass_kg="$(arg wastewater_load_mass_kg)"/>
+  <xacro:hf_product_bodywork parent="base_link" visible="$(arg bodywork_visible)"/>
   <xacro:hf_formal_ros2_control use_sim="$(arg use_sim)"/>
   <xacro:if value="$(arg use_sim)">

File: starter_ws/src/sanitation_vehicle_description/urdf/high_fidelity/a300_platform.xacro (robot description, xacro)
@@ -97,14 +97,15 @@
         <material name="mast_black"><color rgba="0.06 0.07 0.08 1"/></material>
       </visual>
-      <collision name="mast_column_collision"><origin xyz="0 0 0.360"/><geometry><box size="0.060 0.060 0.720"/></geometry></collision>
+      <collision name="mast_column_collision"><origin xyz="0 0 0.425"/><geometry><box size="0.060 0.060 0.850"/></geometry></collision>
       <collision name="mast_crossbar_collision">
-        <origin xyz="0 0 0.700"/>
-        <geometry><box size="0.090 0.480 0.040"/></geometry>
+        <origin xyz="0 0 0.815"/>
+        <geometry><box size="0.090 0.300 0.055"/></geometry>
       </collision>
+      <collision name="mast_gnss_stanchion_collision"><origin xyz="-0.100 0 0.895"/><geometry><box size="0.040 0.040 0.130"/></geometry></collision>
       <collision name="mast_gusset_collision"><origin xyz="0 0 0.060"/><geometry><box size="0.170 0.120 0.120"/></geometry></collision>
       <inertial>
-        <origin xyz="0 0 0.360"/>
+        <origin xyz="0 0 0.425"/>
         <mass value="1.0"/>
-        <xacro:hf_box_inertia mass="1.0" x="0.060" y="0.060" z="0.720"/>
+        <xacro:hf_box_inertia mass="1.0" x="0.060" y="0.060" z="0.850"/>
       </inertial>
     </link>
@@ -119,9 +120,9 @@
         <material name="arm_mount_gray"><color rgba="0.32 0.34 0.36 1"/></material></visual>
       <collision><origin xyz="0 0 0.013"/><geometry><cylinder radius="0.120" length="0.056"/></geometry></collision>
-      <inertial><mass value="0.001"/><inertia ixx="0.000001" ixy="0" ixz="0" iyy="0.000001" iyz="0" izz="0.000001"/></inertial>
+      <inertial><origin xyz="0 0 0.013"/><mass value="2.8"/><inertia ixx="0.010811" ixy="0" ixz="0" iyy="0.010811" iyz="0" izz="0.020160"/></inertial>
     </link>
     <joint name="arm_mount_joint" type="fixed">
       <parent link="payload_deck_link"/><child link="arm_mount_link"/>
-      <origin xyz="0.035 -0.145 0.065"/>
+      <origin xyz="0.100 -0.200 0.065"/>
     </joint>
     <!-- UR e-Series standard control box.  The public cabinet envelope is

File: starter_ws/src/sanitation_vehicle_description/urdf/high_fidelity/cleaning_mechanism.xacro (robot description, xacro)
@@ -322,6 +322,8 @@
       <origin xyz="0.040 0 0.010" rpy="0 0 0"/>
     </joint>
-    <!-- Segmented hose geometry reserves a 50 mm ID flow path while keeping a
-         tree topology. A later fluid plugin binds inlet/outlet coupling frames. -->
+    <!-- Segmented hose geometry reserves a 50 mm ID flow path.  The three
+         centres follow one continuous rising route from the rear nozzle into
+         the enclosed pump bay; explicit chassis-relative mounts avoid the
+         cumulative transform gap that made the upper segment appear detached. -->
     <xacro:macro name="hf_hose_segment" params="name parent xyz rpy length mass mesh">
       <link name="${name}_link">
@@ -332,7 +334,7 @@
       <joint name="${name}_joint" type="fixed"><parent link="${parent}"/><child link="${name}_link"/><origin xyz="${xyz}" rpy="${rpy}"/></joint>
     </xacro:macro>
-    <xacro:hf_hose_segment name="recovery_hose_lower" parent="suction_nozzle_link" xyz="-0.08 0 0.10" rpy="0 -0.58 0" length="0.22" mass="0.140" mesh="recovery_hose_220.stl"/>
-    <xacro:hf_hose_segment name="recovery_hose_middle" parent="recovery_hose_lower_link" xyz="-0.16 0 0.10" rpy="0 -0.70 0" length="0.25" mass="0.160" mesh="recovery_hose_250.stl"/>
-    <xacro:hf_hose_segment name="recovery_hose_upper" parent="recovery_hose_middle_link" xyz="-0.17 0 0.14" rpy="0 -0.35 0" length="0.20" mass="0.120" mesh="recovery_hose_200.stl"/>
+    <xacro:hf_hose_segment name="recovery_hose_lower" parent="cleaning_mechanism_mount_link" xyz="-0.470 0 0.100" rpy="0 -0.750 0" length="0.22" mass="0.140" mesh="recovery_hose_220.stl"/>
+    <xacro:hf_hose_segment name="recovery_hose_middle" parent="cleaning_mechanism_mount_link" xyz="-0.320 0 0.280" rpy="0 -0.950 0" length="0.25" mass="0.160" mesh="recovery_hose_250.stl"/>
+    <xacro:hf_hose_segment name="recovery_hose_upper" parent="cleaning_mechanism_mount_link" xyz="-0.202 0 0.471" rpy="0 -1.100 0" length="0.20" mass="0.120" mesh="recovery_hose_200.stl"/>
     <link name="recovery_strainer_filter_link">
       <xacro:hf_clean_visual mesh="strainer_filter_bowl.stl"

File: starter_ws/src/sanitation_vehicle_description/urdf/high_fidelity/manipulator_stack.xacro (robot description, xacro)
@@ -20,5 +20,5 @@
          the seven physical UR links retain the published 20.6 kg total. -->
     <link name="ur5e_base_link"/>
-    <joint name="ur5e_mount_joint" type="fixed"><parent link="${parent}"/><child link="ur5e_base_link"/><origin xyz="0 0 0.015"/></joint>
+    <joint name="ur5e_mount_joint" type="fixed"><parent link="${parent}"/><child link="ur5e_base_link"/><origin xyz="0 0 0.045"/></joint>
     <!-- The official UR description separates the REP-103 base frame from the
          controller-facing inertial frame with a pi rotation. The mesh itself

File: starter_ws/src/sanitation_vehicle_description/urdf/high_fidelity/sensor_suite.xacro (robot description, xacro)
@@ -100,6 +100,6 @@
       <inertial><origin xyz="0 0 -0.0115"/><mass value="0.37"/><xacro:hf_sensor_box_inertia mass="0.37" x="0.060" y="0.060" z="0.087"/></inertial>
     </link>
-    <joint name="lidar_2d_mount_joint" type="fixed"><parent link="${mast_parent}"/><child link="lidar_2d_link"/>
-      <origin xyz="0.380 0 0.395"/></joint>
+    <joint name="lidar_2d_mount_joint" type="fixed"><parent link="${base_parent}"/><child link="lidar_2d_link"/>
+      <origin xyz="0.250 0 0.665"/></joint>
     <gazebo reference="lidar_2d_link">
       <sensor name="utm30lx" type="gpu_lidar">
@@ -124,5 +124,5 @@
     </link>
     <joint name="lidar_3d_mount_joint" type="fixed"><parent link="${mast_parent}"/><child link="lidar_3d_link"/>
-      <origin xyz="0 0 0.725"/></joint>
+      <origin xyz="0 0 0.845"/></joint>
     <gazebo reference="lidar_3d_link">
       <sensor name="mid360" type="gpu_lidar">
@@ -135,5 +135,5 @@
       </sensor>
     </gazebo>
-    <xacro:hf_d435 name="front_rgbd" parent="${mast_parent}" xyz="0.640 0 0.225" rpy="0 0 0"
+    <xacro:hf_d435 name="front_rgbd" parent="${base_parent}" xyz="0.570 0 0.449" rpy="0 0 0"
                     topic="/sensors/front_rgbd/depth/image_rect_raw" max_range="10.0"/>
     <!-- Side bracket position keeps the camera outside the Robotiq base and
@@ -142,9 +142,9 @@
                     topic="/sensors/wrist_rgbd/depth/image_rect_raw" max_range="3.0" mount_bracket="true"/>
     <!-- Independent modules: each has its own housing, imager, frame and topic. -->
-    <xacro:hf_fisheye name="rear_left_fisheye" parent="${mast_parent}" xyz="-0.350 0.275 0.200" rpy="0 -0.175 2.705"
+    <xacro:hf_fisheye name="rear_left_fisheye" parent="${base_parent}" xyz="-0.565 0.280 0.435" rpy="0 -0.175 2.705"
                        optical_xyz="0.022011096607 -0.000604893394 -0.003891751553"
                        optical_rpy="-1.745999996444 -0.000035461162 -1.570996889205"
                        topic="/sensors/rear_left_fisheye/image_raw"/>
-    <xacro:hf_fisheye name="rear_right_fisheye" parent="${mast_parent}" xyz="-0.350 -0.275 0.200" rpy="0 -0.175 -2.705"
+    <xacro:hf_fisheye name="rear_right_fisheye" parent="${base_parent}" xyz="-0.565 -0.280 0.435" rpy="0 -0.175 -2.705"
                        optical_xyz="0.022011096607 0.000604893394 -0.003891751553"
                        optical_rpy="-1.745999996444 -0.000035461162 -1.570996889205"
@@ -158,5 +158,5 @@
     </link>
     <joint name="gnss_antenna_mount_joint" type="fixed"><parent link="${mast_parent}"/><child link="gnss_antenna_link"/>
-      <origin xyz="0 0 0.845"/></joint>
+      <origin xyz="-0.100 0 0.965"/></joint>
     <gazebo reference="gnss_antenna_link">
       <sensor name="zed_f9p" type="navsat"><topic>/sensors/gnss/fix</topic><update_rate>10</update_rate>
