Commit message: feat: finalize sensor tower and manipulator simulation

File: reports/engineering/formal_competition_vehicle.urdf (robot description, URDF)
Before this commit: robot tzcup_formal_sanitation_vehicle, 115 links, 114 joints
Links:
- added link front_rgbd_mount_link, mass 0.18; collision box size=0.045 0.008 0.052; collision box size=0.045 0.008 0.052
- added link gnss_mount_link, mass 0.24; collision box size=0.100 0.230 0.018; collision cylinder length=0.002 radius=0.075
- added link imu_mount_tray_link, mass 0.12; collision box size=0.090 0.080 0.022; visual mesh filename=package://sanitation_vehicle_description/meshes/generated/p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
- added link lidar_2d_mount_link, mass 0.42; collision box size=0.014 0.105 0.090; collision box size=0.100 0.090 0.008
- added link lidar_3d_mount_link, mass 0.28; collision cylinder length=0.034 radius=0.070; visual mesh filename=package://sanitation_vehicle_description/meshes/generated/p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
- added link rear_left_fisheye_mount_link, mass 0.14; collision box size=0.020 0.090 0.084; collision box size=0.028 0.074 0.008
- added link rear_right_fisheye_mount_link, mass 0.14; collision box size=0.020 0.090 0.084; collision box size=0.028 0.074 0.008
- link arm_mount_link: mass 2.8 -> 6.5; geometry collision box size=0.180 0.180 0.040; collision box size=0.280 0.220 0.012
- link bodywork_rear_shell_link: geometry collision box size=0.13 0.15 0.35; collision box size=0.53 0.70 0.52
- link gnss_antenna_link: mass 0.10 -> 0.173
- link sensor_mast_link: mass 1.0 -> 1.45; geometry collision box size=0.030 0.030 0.760; collision box size=0.030 0.030 0.760
Joints:
- added joint front_rgbd_bracket_joint: type fixed, parent base_link, child front_rgbd_mount_link, origin xyz=0.565 0 0.449 rpy=0 0.139626 0
- added joint gnss_bracket_joint: type fixed, parent sensor_mast_link, child gnss_mount_link, origin xyz=-0.035 -0.020 0.765
- added joint imu_tray_joint: type fixed, parent base_link, child imu_mount_tray_link, origin xyz=0 0 0.225
- added joint lidar_2d_bracket_joint: type fixed, parent sensor_mast_link, child lidar_2d_mount_link, origin xyz=0.060 0 0.635
- added joint lidar_3d_bracket_joint: type fixed, parent sensor_mast_link, child lidar_3d_mount_link, origin xyz=0 0 0.790
- added joint rear_left_fisheye_bracket_joint: type fixed, parent base_link, child rear_left_fisheye_mount_link, origin xyz=-0.565 0.280 0.435 rpy=0 -0.175 2.705
- added joint rear_right_fisheye_bracket_joint: type fixed, parent base_link, child rear_right_fisheye_mount_link, origin xyz=-0.565 -0.280 0.435 rpy=0 -0.175 -2.705
- joint front_rgbd_mount_joint: origin xyz=0.570 0 0.449 rpy=0 0 0 -> xyz=0.005 0 0 rpy=0 0 0; parent base_link -> front_rgbd_mount_link
- joint gnss_antenna_mount_joint: origin xyz=-0.100 0 0.965 -> xyz=-0.020 0.180 0.026; parent sensor_mast_link -> gnss_mount_link
- joint imu_mount_joint: origin xyz=0 0 0.244 -> xyz=0 0 0.019; parent base_link -> imu_mount_tray_link
- joint lidar_2d_mount_joint: origin xyz=0.250 0 0.665 -> xyz=0.055 0 0.078; parent base_link -> lidar_2d_mount_link
- joint lidar_3d_mount_joint: origin xyz=0 0 0.845 -> xyz=0 0 0.094; parent sensor_mast_link -> lidar_3d_mount_link
- joint rear_left_fisheye_mount_joint: origin xyz=-0.565 0.280 0.435 rpy=0 -0.175 2.705 -> xyz=0 0 0 rpy=0 0 0; parent base_link -> rear_left_fisheye_mount_link
- joint rear_right_fisheye_mount_joint: origin xyz=-0.565 -0.280 0.435 rpy=0 -0.175 -2.705 -> xyz=0 0 0 rpy=0 0 0; parent base_link -> rear_right_fisheye_mount_link

File: starter_ws/src/sanitation_vehicle_description/urdf/high_fidelity/a300_platform.xacro (robot description, xacro)
@@ -90,22 +90,21 @@
       <origin xyz="0 0 0.204"/>
     </joint>
-    <!-- Structural mast is intentionally a separate physical link so its
-         flexibility and sensor payload can be refined without changing base inertia. -->
+    <!-- Bolted twin-column sensor tower.  Sensor-specific shelves are separate
+         physical links in sensor_suite.xacro, so every load path is visible
+         and no sensor is represented as floating on an anonymous crossbar. -->
     <link name="sensor_mast_link">
       <visual name="machined_sensor_mast_visual">
         <geometry><mesh filename="package://sanitation_vehicle_description/meshes/generated/platform/sensor_mast.stl"/></geometry>
-        <material name="mast_black"><color rgba="0.06 0.07 0.08 1"/></material>
+        <material name="mast_anodized_aluminum"><color rgba="0.30 0.33 0.34 1"/></material>
       </visual>
-      <collision name="mast_column_collision"><origin xyz="0 0 0.425"/><geometry><box size="0.060 0.060 0.850"/></geometry></collision>
-      <collision name="mast_crossbar_collision">
-        <origin xyz="0 0 0.815"/>
-        <geometry><box size="0.090 0.300 0.055"/></geometry>
-      </collision>
-      <collision name="mast_gnss_stanchion_collision"><origin xyz="-0.100 0 0.895"/><geometry><box size="0.040 0.040 0.130"/></geometry></collision>
-      <collision name="mast_gusset_collision"><origin xyz="0 0 0.060"/><geometry><box size="0.170 0.120 0.120"/></geometry></collision>
+      <collision name="mast_left_column_collision"><origin xyz="0 -0.050 0.396"/><geometry><box size="0.030 0.030 0.760"/></geometry></collision>
+      <collision name="mast_right_column_collision"><origin xyz="0 0.050 0.396"/><geometry><box size="0.030 0.030 0.760"/></geometry></collision>
+      <collision name="mast_service_spine_collision"><origin xyz="-0.022 0 0.375"/><geometry><box size="0.036 0.062 0.690"/></geometry></collision>
+      <collision name="mast_pedestal_collision"><origin xyz="0 0 0.008"/><geometry><box size="0.190 0.150 0.016"/></geometry></collision>
+      <collision name="mast_head_plate_collision"><origin xyz="0 0 0.778"/><geometry><box size="0.150 0.120 0.018"/></geometry></collision>
       <inertial>
-        <origin xyz="0 0 0.425"/>
-        <mass value="1.0"/>
-        <xacro:hf_box_inertia mass="1.0" x="0.060" y="0.060" z="0.850"/>
+        <origin xyz="0 0 0.390"/>
+        <mass value="1.45"/>
+        <xacro:hf_box_inertia mass="1.45" x="0.150" y="0.150" z="0.780"/>
       </inertial>
     </link>
@@ -119,6 +118,8 @@
       <visual><geometry><mesh filename="package://sanitation_vehicle_description/meshes/generated/platform/arm_mount_adapter.stl"/></geometry>
         <material name="arm_mount_gray"><color rgba="0.32 0.34 0.36 1"/></material></visual>
-      <collision><origin xyz="0 0 0.013"/><geometry><cylinder radius="0.120" length="0.056"/></geometry></collision>
-      <inertial><origin xyz="0 0 0.013"/><mass value="2.8"/><inertia ixx="0.010811" ixy="0" ixz="0" iyy="0.010811" iyz="0" izz="0.020160"/></inertial>
+      <collision name="arm_backing_plate_collision"><origin xyz="0 0 -0.044"/><geometry><box size="0.280 0.220 0.012"/></geometry></collision>
+      <collision name="arm_pedestal_collision"><origin xyz="0 0 -0.018"/><geometry><box size="0.180 0.180 0.040"/></geometry></collision>
+      <collision name="arm_adapter_collision"><origin xyz="0 0 0.013"/><geometry><cylinder radius="0.120" length="0.056"/></geometry></collision>
+      <inertial><origin xyz="0 0 -0.005"/><mass value="6.5"/><inertia ixx="0.035100" ixy="0" ixz="0" iyy="0.035100" iyz="0" izz="0.048100"/></inertial>
     </link>
     <joint name="arm_mount_joint" type="fixed">

File: starter_ws/src/sanitation_vehicle_description/urdf/high_fidelity/bodywork.xacro (robot description, xacro)
@@ -96,4 +96,5 @@
       <xacro:hf_body_visual mesh="rear_bin_outer_shell.stl" material="body_warm_white" rgba="0.86 0.89 0.88 1" visible="${visible}"/>
       <xacro:hf_body_visual mesh="sensor_pylon_fairing.stl" material="sensor_pylon" rgba="0.070 0.085 0.088 1" visible="${visible}"/>
+      <xacro:hf_body_visual mesh="sensor_pylon_service_hatch.stl" material="sensor_pylon_hatch" rgba="0.16 0.18 0.19 1" visible="${visible}"/>
       <collision name="rear_shell_collision"><origin xyz="-0.285 0 0.495"/><geometry><box size="0.53 0.70 0.52"/></geometry></collision>
       <collision name="pylon_fairing_collision"><origin xyz="-0.135 0 0.770"/><geometry><box size="0.13 0.15 0.35"/></geometry></collision>

File: starter_ws/src/sanitation_vehicle_description/urdf/high_fidelity/sensor_suite.xacro (robot description, xacro)
@@ -56,5 +56,8 @@
           <image><width>848</width><height>480</height><format>R8G8B8</format></image>
           <clip><near>0.2</near><far>${max_range}</far></clip>
-          <lens><intrinsics><fx>430.0</fx><fy>430.0</fy><cx>424.0</cx><cy>240.0</cy><s>0</s></intrinsics></lens>
+          <!-- Intrinsics are internally consistent with the 87 x 58 degree
+               D435 envelope at 848 x 480; deployment replaces these with the
+               serial-number-specific calibration. -->
+          <lens><intrinsics><fx>447.2</fx><fy>433.0</fy><cx>424.0</cx><cy>240.0</cy><s>0</s></intrinsics></lens>
           <depth_camera><output>depths</output></depth_camera>
         </camera>
@@ -94,12 +97,26 @@
   </xacro:macro>
   <xacro:macro name="hf_sensor_suite" params="mast_parent base_parent wrist_parent">
+    <!-- Every fixed sensor is connected through a named, physical mounting
+         link.  This makes the installation hierarchy inspectable in TF/URDF
+         and keeps the visible vendor housing separate from project-owned CAD. -->
     <!-- Hokuyo UTM-30LX: 60 x 60 x 87 mm, 0.37 kg, 270 deg at 40 Hz. -->
+    <link name="lidar_2d_mount_link">
+      <visual name="utm30lx_bracket_visual"><geometry><mesh filename="package://sanitation_vehicle_description/meshes/generated/platform/utm30lx_mount.stl"/></geometry>
+        <material name="sensor_mount_silver"><color rgba="0.42 0.46 0.47 1"/></material></visual>
+      <collision name="utm_shelf_collision"><origin xyz="0.020 0 0.006"/><geometry><box size="0.150 0.120 0.014"/></geometry></collision>
+      <collision name="utm_backplate_collision"><origin xyz="-0.048 0 -0.030"/><geometry><box size="0.014 0.105 0.090"/></geometry></collision>
+      <collision name="utm_pad_collision"><origin xyz="0.055 0 0.019"/><geometry><box size="0.100 0.090 0.008"/></geometry></collision>
+      <inertial><mass value="0.42"/><xacro:hf_sensor_box_inertia mass="0.42" x="0.150" y="0.120" z="0.110"/></inertial>
+    </link>
+    <joint name="lidar_2d_bracket_joint" type="fixed"><parent link="${mast_parent}"/><child link="lidar_2d_mount_link"/>
+      <origin xyz="0.060 0 0.635"/></joint>
     <link name="lidar_2d_link">
-      <visual name="utm30lx_mesh"><geometry><mesh filename="package://sanitation_vehicle_description/meshes/vendor/robotnik_sensors/hokuyo_utm_30lx.dae"/></geometry></visual>
+      <visual name="utm30lx_mesh"><geometry><mesh filename="package://sanitation_vehicle_description/meshes/vendor/robotnik_sensors/hokuyo_utm_30lx.dae"/></geometry>
+        <material name="utm30lx_blue"><color rgba="0.08 0.29 0.44 1"/></material></visual>
       <collision><origin xyz="0 0 -0.0115"/><geometry><box size="0.060 0.060 0.087"/></geometry></collision>
       <inertial><origin xyz="0 0 -0.0115"/><mass value="0.37"/><xacro:hf_sensor_box_inertia mass="0.37" x="0.060" y="0.060" z="0.087"/></inertial>
     </link>
-    <joint name="lidar_2d_mount_joint" type="fixed"><parent link="${base_parent}"/><child link="lidar_2d_link"/>
-      <origin xyz="0.250 0 0.665"/></joint>
+    <joint name="lidar_2d_mount_joint" type="fixed"><parent link="lidar_2d_mount_link"/><child link="lidar_2d_link"/>
+      <origin xyz="0.055 0 0.078"/></joint>
     <gazebo reference="lidar_2d_link">
       <sensor name="utm30lx" type="gpu_lidar">
@@ -113,4 +130,12 @@
     </gazebo>
     <!-- Livox MID-360 physical envelope and non-repeating scan approximation. -->
+    <link name="lidar_3d_mount_link">
+      <visual name="mid360_isolator_plate_visual"><geometry><mesh filename="package://sanitation_vehicle_description/meshes/generated/platform/mid360_mount.stl"/></geometry>
+        <material name="mid360_mount_silver"><color rgba="0.48 0.52 0.53 1"/></material></visual>
+      <collision><origin xyz="0 0 0.017"/><geometry><cylinder radius="0.070" length="0.034"/></geometry></collision>
+      <inertial><origin xyz="0 0 0.017"/><mass value="0.28"/><inertia ixx="0.000360" ixy="0" ixz="0" iyy="0.000360" iyz="0" izz="0.000686"/></inertial>
+    </link>
+    <joint name="lidar_3d_bracket_joint" type="fixed"><parent link="${mast_parent}"/><child link="lidar_3d_mount_link"/>
+      <origin xyz="0 0 0.790"/></joint>
     <link name="lidar_3d_link">
       <visual name="mid360_mesh">
@@ -119,10 +144,11 @@
         <origin xyz="0 0 -0.0365" rpy="${pi/2.0} 0 0"/>
         <geometry><mesh filename="package://sanitation_vehicle_description/meshes/vendor/robotnik_sensors/livox_mid_360.stl" scale="0.001 0.001 0.001"/></geometry>
+        <material name="mid360_dark_gray"><color rgba="0.11 0.13 0.14 1"/></material>
       </visual>
       <collision><origin xyz="0 0 -0.0325"/><geometry><cylinder radius="0.041" length="0.060"/></geometry></collision>
       <inertial><origin xyz="0 0 -0.0325"/><mass value="0.265"/><inertia ixx="0.000103" ixy="0" ixz="0" iyy="0.000103" iyz="0" izz="0.000140"/></inertial>
     </link>
-    <joint name="lidar_3d_mount_joint" type="fixed"><parent link="${mast_parent}"/><child link="lidar_3d_link"/>
-      <origin xyz="0 0 0.845"/></joint>
+    <joint name="lidar_3d_mount_joint" type="fixed"><parent link="lidar_3d_mount_link"/><child link="lidar_3d_link"/>
+      <origin xyz="0 0 0.094"/></joint>
     <gazebo reference="lidar_3d_link">
       <sensor name="mid360" type="gpu_lidar">
@@ -130,10 +156,22 @@
         <gz_frame_id>lidar_3d_link</gz_frame_id>
         <lidar><scan><horizontal><samples>1800</samples><resolution>1</resolution><min_angle>-${pi}</min_angle><max_angle>${pi}</max_angle></horizontal>
-          <vertical><samples>64</samples><resolution>1</resolution><min_angle>-0.514872</min_angle><max_angle>0.514872</max_angle></vertical></scan>
+          <!-- MID-360 published vertical field of view: -7 to +52 degrees. -->
+          <vertical><samples>64</samples><resolution>1</resolution><min_angle>-0.122173</min_angle><max_angle>0.907571</max_angle></vertical></scan>
           <range><min>0.1</min><max>40.0</max><resolution>0.01</resolution></range>
           <noise><type>gaussian</type><mean>0</mean><stddev>0.020</stddev></noise></lidar>
       </sensor>
     </gazebo>
-    <xacro:hf_d435 name="front_rgbd" parent="${base_parent}" xyz="0.570 0 0.449" rpy="0 0 0"
+    <link name="front_rgbd_mount_link">
+      <visual name="front_rgbd_bezel_visual"><geometry><mesh filename="package://sanitation_vehicle_description/meshes/generated/platform/front_rgbd_mount.stl"/></geometry>
+        <material name="front_rgbd_bezel"><color rgba="0.055 0.070 0.073 1"/></material></visual>
+      <collision name="front_rgbd_upper_bezel"><origin xyz="0 0 0.030"/><geometry><box size="0.045 0.132 0.008"/></geometry></collision>
+      <collision name="front_rgbd_lower_bezel"><origin xyz="0 0 -0.030"/><geometry><box size="0.045 0.132 0.008"/></geometry></collision>
+      <collision name="front_rgbd_left_bezel"><origin xyz="0 0.062 0"/><geometry><box size="0.045 0.008 0.052"/></geometry></collision>
+      <collision name="front_rgbd_right_bezel"><origin xyz="0 -0.062 0"/><geometry><box size="0.045 0.008 0.052"/></geometry></collision>
+      <inertial><mass value="0.18"/><xacro:hf_sensor_box_inertia mass="0.18" x="0.045" y="0.132" z="0.067"/></inertial>
+    </link>
+    <joint name="front_rgbd_bracket_joint" type="fixed"><parent link="${base_parent}"/><child link="front_rgbd_mount_link"/>
+      <origin xyz="0.565 0 0.449" rpy="0 0.139626 0"/></joint>
+    <xacro:hf_d435 name="front_rgbd" parent="front_rgbd_mount_link" xyz="0.005 0 0" rpy="0 0 0"
                     topic="/sensors/front_rgbd/depth/image_rect_raw" max_range="10.0"/>
     <!-- Side bracket position keeps the camera outside the Robotiq base and
@@ -142,21 +180,45 @@
                     topic="/sensors/wrist_rgbd/depth/image_rect_raw" max_range="3.0" mount_bracket="true"/>
     <!-- Independent modules: each has its own housing, imager, frame and topic. -->
-    <xacro:hf_fisheye name="rear_left_fisheye" parent="${base_parent}" xyz="-0.565 0.280 0.435" rpy="0 -0.175 2.705"
+    <link name="rear_left_fisheye_mount_link">
+      <visual><geometry><mesh filename="package://sanitation_vehicle_description/meshes/generated/platform/rear_fisheye_mount.stl"/></geometry><material name="rear_camera_pod"><color rgba="0.055 0.070 0.073 1"/></material></visual>
+      <collision name="rear_left_pod_back"><origin xyz="-0.018 0 0"/><geometry><box size="0.020 0.090 0.084"/></geometry></collision>
+      <collision name="rear_left_pod_top"><origin xyz="0.004 0 0.038"/><geometry><box size="0.028 0.074 0.008"/></geometry></collision>
+      <collision name="rear_left_pod_bottom"><origin xyz="0.004 0 -0.038"/><geometry><box size="0.028 0.074 0.008"/></geometry></collision>
+      <inertial><mass value="0.14"/><xacro:hf_sensor_box_inertia mass="0.14" x="0.048" y="0.090" z="0.084"/></inertial>
+    </link>
+    <joint name="rear_left_fisheye_bracket_joint" type="fixed"><parent link="${base_parent}"/><child link="rear_left_fisheye_mount_link"/><origin xyz="-0.565 0.280 0.435" rpy="0 -0.175 2.705"/></joint>
+    <xacro:hf_fisheye name="rear_left_fisheye" parent="rear_left_fisheye_mount_link" xyz="0 0 0" rpy="0 0 0"
                        optical_xyz="0.022011096607 -0.000604893394 -0.003891751553"
                        optical_rpy="-1.745999996444 -0.000035461162 -1.570996889205"
                        topic="/sensors/rear_left_fisheye/image_raw"/>
-    <xacro:hf_fisheye name="rear_right_fisheye" parent="${base_parent}" xyz="-0.565 -0.280 0.435" rpy="0 -0.175 -2.705"
+    <link name="rear_right_fisheye_mount_link">
+      <visual><geometry><mesh filename="package://sanitation_vehicle_description/meshes/generated/platform/rear_fisheye_mount.stl"/></geometry><material name="rear_camera_pod_right"><color rgba="0.055 0.070 0.073 1"/></material></visual>
+      <collision name="rear_right_pod_back"><origin xyz="-0.018 0 0"/><geometry><box size="0.020 0.090 0.084"/></geometry></collision>
+      <collision name="rear_right_pod_top"><origin xyz="0.004 0 0.038"/><geometry><box size="0.028 0.074 0.008"/></geometry></collision>
+      <collision name="rear_right_pod_bottom"><origin xyz="0.004 0 -0.038"/><geometry><box size="0.028 0.074 0.008"/></geometry></collision>
+      <inertial><mass value="0.14"/><xacro:hf_sensor_box_inertia mass="0.14" x="0.048" y="0.090" z="0.084"/></inertial>
+    </link>
+    <joint name="rear_right_fisheye_bracket_joint" type="fixed"><parent link="${base_parent}"/><child link="rear_right_fisheye_mount_link"/><origin xyz="-0.565 -0.280 0.435" rpy="0 -0.175 -2.705"/></joint>
+    <xacro:hf_fisheye name="rear_right_fisheye" parent="rear_right_fisheye_mount_link" xyz="0 0 0" rpy="0 0 0"
                        optical_xyz="0.022011096607 0.000604893394 -0.003891751553"
                        optical_rpy="-1.745999996444 -0.000035461162 -1.570996889205"
                        topic="/sensors/rear_right_fisheye/image_raw"/>
-    <!-- ZED-F9P receiver mass is represented together with ANN-MB-00 antenna. -->
+    <!-- ANN-MB GNSS antenna sits on a dedicated side boom so the MID-360 has
+         an unobstructed 360-degree crown and the antenna retains sky view. -->
+    <link name="gnss_mount_link">
+      <visual><geometry><mesh filename="package://sanitation_vehicle_description/meshes/generated/platform/gnss_mount.stl"/></geometry><material name="gnss_mount_silver"><color rgba="0.45 0.49 0.50 1"/></material></visual>
+      <collision name="gnss_boom_collision"><origin xyz="0 0.085 0"/><geometry><box size="0.100 0.230 0.018"/></geometry></collision>
+      <collision name="gnss_ground_plane_collision"><origin xyz="-0.020 0.180 0.010"/><geometry><cylinder radius="0.075" length="0.002"/></geometry></collision>
+      <inertial><origin xyz="0 0.085 0"/><mass value="0.24"/><xacro:hf_sensor_box_inertia mass="0.24" x="0.100" y="0.230" z="0.073"/></inertial>
+    </link>
+    <joint name="gnss_bracket_joint" type="fixed"><parent link="${mast_parent}"/><child link="gnss_mount_link"/><origin xyz="-0.035 -0.020 0.765"/></joint>
     <link name="gnss_antenna_link">
       <visual name="ann_mb_mesh"><origin xyz="0 0 -0.01125"/>
         <geometry><mesh filename="package://sanitation_vehicle_description/meshes/vendor/robotnik_sensors/antenna_ANN_MB.stl"/></geometry></visual>
       <collision><geometry><box size="0.0607 0.083 0.0225"/></geometry></collision>
-      <inertial><mass value="0.10"/><inertia ixx="0.000026" ixy="0" ixz="0" iyy="0.000026" iyz="0" izz="0.000045"/></inertial>
-    </link>
-    <joint name="gnss_antenna_mount_joint" type="fixed"><parent link="${mast_parent}"/><child link="gnss_antenna_link"/>
-      <origin xyz="-0.100 0 0.965"/></joint>
+      <inertial><mass value="0.173"/><inertia ixx="0.000091" ixy="0" ixz="0" iyy="0.000060" iyz="0" izz="0.000130"/></inertial>
+    </link>
+    <joint name="gnss_antenna_mount_joint" type="fixed"><parent link="gnss_mount_link"/><child link="gnss_antenna_link"/>
+      <origin xyz="-0.020 0.180 0.026"/></joint>
     <gazebo reference="gnss_antenna_link">
       <sensor name="zed_f9p" type="navsat"><topic>/sensors/gnss/fix</topic><update_rate>10</update_rate>
@@ -168,5 +230,11 @@
       </sensor>
     </gazebo>
-    <!-- VN-100 Rugged body is located near the vehicle CoG, not on the mast. -->
+    <!-- VN-100 Rugged body is internally isolated near the vehicle CoG. -->
+    <link name="imu_mount_tray_link">
+      <visual><geometry><mesh filename="package://sanitation_vehicle_description/meshes/generated/platform/imu_mount_tray.stl"/></geometry><material name="imu_tray"><color rgba="0.40 0.44 0.45 1"/></material></visual>
+      <collision><origin xyz="0 0 0.008"/><geometry><box size="0.090 0.080 0.022"/></geometry></collision>
+      <inertial><origin xyz="0 0 0.008"/><mass value="0.12"/><xacro:hf_sensor_box_inertia mass="0.12" x="0.090" y="0.080" z="0.022"/></inertial>
+    </link>
+    <joint name="imu_tray_joint" type="fixed"><parent link="${base_parent}"/><child link="imu_mount_tray_link"/><origin xyz="0 0 0.225"/></joint>
     <link name="imu_link">
       <!-- Invert Robotnik's base-to-measurement-frame offset so imu_link
@@ -177,6 +245,6 @@
       <inertial><origin xyz="0.00745 0 -0.0043"/><mass value="0.015"/><xacro:hf_sensor_box_inertia mass="0.015" x="0.036" y="0.037" z="0.009"/></inertial>
     </link>
-    <joint name="imu_mount_joint" type="fixed"><parent link="${base_parent}"/><child link="imu_link"/>
-      <origin xyz="0 0 0.244"/></joint>
+    <joint name="imu_mount_joint" type="fixed"><parent link="imu_mount_tray_link"/><child link="imu_link"/>
+      <origin xyz="0 0 0.019"/></joint>
     <gazebo reference="imu_link">
       <sensor name="vn100" type="imu"><topic>/sensors/imu/data</topic><update_rate>200</update_rate><always_on>true</always_on>
