Commit message: feat(vehicle): complete formal sanitation function layout

File: reports/engineering/formal_competition_vehicle.urdf (robot description, URDF)
Before this commit: robot tzcup_formal_sanitation_vehicle, 122 links, 121 joints
Links:
- added link dry_deposit_chute_link, mass 0.32; collision box size=0.125 0.100 0.350; visual mesh filename=package://sanitation_vehicle_description/meshes/project/sto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
- added link dry_deposit_gate_link, mass 0.18; collision box size=0.184 0.158 0.008; visual mesh filename=package://sanitation_vehicle_description/meshes/project/sto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
- added link dry_deposit_hopper_link, mass 0.24; collision box size=0.010 0.165 0.092; collision box size=0.010 0.165 0.092
- added link dry_deposit_presence_sensor_link, mass 0.045; collision box size=0.040 0.055 0.022; visual mesh filename=package://sanitation_vehicle_description/meshes/project/sto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
- added link isolated_dc_dc_module_link, mass 0.400; collision box size=0.140 0.100 0.055; visual mesh filename=package://sanitation_vehicle_description/meshes/generated/p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
- added link power_distribution_box_link, mass 0.700; collision box size=0.190 0.125 0.068; visual mesh filename=package://sanitation_vehicle_description/meshes/generated/p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
- added link recovery_flow_sensor_link, mass 0.22; collision box size=0.070 0.105 0.075; visual mesh filename=package://sanitation_vehicle_description/meshes/project/cle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
- added link recovery_pump_rotor_link, mass 0.12; collision cylinder length=0.018 radius=0.035; visual mesh filename=package://sanitation_vehicle_description/meshes/project/cle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
- added link safety_relay_link, mass 0.250; collision box size=0.110 0.080 0.065; visual mesh filename=package://sanitation_vehicle_description/meshes/generated/p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
- link bodywork_rear_shell_link: geometry collision box size=0.045 0.70 0.52; collision box size=0.080 0.270 0.055
- link dry_bin_lid_link: geometry collision box size=0.179 0.181 0.010; collision box size=0.179 0.181 0.010
Joints:
- added joint dry_deposit_chute_mount_joint: type fixed, parent dry_deposit_hopper_link, child dry_deposit_chute_link, origin xyz=0 0 -0.180 rpy=0 0 0
- added joint dry_deposit_gate_joint: type revolute, parent dry_deposit_hopper_link, child dry_deposit_gate_link, origin xyz=-0.095 0 0.044 rpy=0 0 0, axis 0 1 0, limit lower=0.0 upper=1.75 effort=22.0 velocity=0.8
- added joint dry_deposit_hopper_mount_joint: type fixed, parent dry_bin_lid_link, child dry_deposit_hopper_link, origin xyz=0.254 0 0.350 rpy=0 0 0
- added joint dry_deposit_presence_sensor_joint: type fixed, parent dry_deposit_hopper_link, child dry_deposit_presence_sensor_link, origin xyz=0.088 0 0.015 rpy=0 0 0
- added joint isolated_dc_dc_mount_joint: type fixed, parent payload_deck_link, child isolated_dc_dc_module_link, origin xyz=0.345 -0.105 0.070
- added joint power_distribution_box_mount_joint: type fixed, parent payload_deck_link, child power_distribution_box_link, origin xyz=0.330 0.025 0.075
- added joint recovery_flow_sensor_mount_joint: type fixed, parent wastewater_delivery_coupling_link, child recovery_flow_sensor_link, origin xyz=0 -0.095 0 rpy=0 0 0
- added joint recovery_pump_joint: type continuous, parent recovery_pump_head_link, child recovery_pump_rotor_link, origin xyz=0 0 0.043 rpy=0 0 0, axis 0 0 1, limit effort=18.0 velocity=62.832
- added joint safety_relay_mount_joint: type fixed, parent payload_deck_link, child safety_relay_link, origin xyz=0.220 -0.080 0.075

File: starter_ws/src/sanitation_vehicle_description/urdf/high_fidelity/a300_platform.xacro (robot description, xacro)
@@ -169,4 +169,37 @@
       <origin xyz="0 0 0"/>
     </joint>
+    <!-- Explicit protected power path: A300 battery/VBAT enters a fused PDU,
+         an isolated converter supplies sensors/compute, and the safety relay
+         removes cleaning/manipulator enable independently of software. -->
+    <link name="power_distribution_box_link">
+      <visual><geometry><mesh filename="package://sanitation_vehicle_description/meshes/generated/platform/power_distribution_box.stl"/></geometry>
+        <material name="pdu_red"><color rgba="0.45 0.055 0.045 1"/></material></visual>
+      <collision><geometry><box size="0.190 0.125 0.068"/></geometry></collision>
+      <inertial><mass value="0.700"/><xacro:hf_box_inertia mass="0.700" x="0.190" y="0.125" z="0.068"/></inertial>
+    </link>
+    <joint name="power_distribution_box_mount_joint" type="fixed">
+      <parent link="payload_deck_link"/><child link="power_distribution_box_link"/>
+      <origin xyz="0.330 0.025 0.075"/>
+    </joint>
+    <link name="isolated_dc_dc_module_link">
+      <visual><geometry><mesh filename="package://sanitation_vehicle_description/meshes/generated/platform/isolated_dc_dc_module.stl"/></geometry>
+        <material name="dc_dc_blue"><color rgba="0.055 0.22 0.36 1"/></material></visual>
+      <collision><geometry><box size="0.140 0.100 0.055"/></geometry></collision>
+      <inertial><mass value="0.400"/><xacro:hf_box_inertia mass="0.400" x="0.140" y="0.100" z="0.055"/></inertial>
+    </link>
+    <joint name="isolated_dc_dc_mount_joint" type="fixed">
+      <parent link="payload_deck_link"/><child link="isolated_dc_dc_module_link"/>
+      <origin xyz="0.345 -0.105 0.070"/>
+    </joint>
+    <link name="safety_relay_link">
+      <visual><geometry><mesh filename="package://sanitation_vehicle_description/meshes/generated/platform/safety_relay.stl"/></geometry>
+        <material name="safety_relay_yellow"><color rgba="0.92 0.58 0.035 1"/></material></visual>
+      <collision><geometry><box size="0.110 0.080 0.065"/></geometry></collision>
+      <inertial><mass value="0.250"/><xacro:hf_box_inertia mass="0.250" x="0.110" y="0.080" z="0.065"/></inertial>
+    </link>
+    <joint name="safety_relay_mount_joint" type="fixed">
+      <parent link="payload_deck_link"/><child link="safety_relay_link"/>
+      <origin xyz="0.220 -0.080 0.075"/>
+    </joint>
     <!-- Current Clearpath A300 wheelbase and tyre-centre track. -->
     <xacro:hf_a300_wheel name="front_left"  side="left"  x="0.256"  y="0.283"/>

File: starter_ws/src/sanitation_vehicle_description/urdf/high_fidelity/bodywork.xacro (robot description, xacro)
@@ -71,4 +71,14 @@
     </link>
     <joint name="bodywork_lower_tub_joint" type="fixed"><parent link="${parent}"/><child link="bodywork_lower_tub_link"/></joint>
+    <gazebo reference="bodywork_lower_tub_link">
+      <sensor name="front_safety_bumper_contact" type="contact">
+        <topic>/safety/front_bumper/contact</topic><update_rate>200</update_rate><always_on>true</always_on>
+        <contact><collision>front_bumper_collision</collision></contact>
+      </sensor>
+      <sensor name="rear_safety_bumper_contact" type="contact">
+        <topic>/safety/rear_bumper/contact</topic><update_rate>200</update_rate><always_on>true</always_on>
+        <contact><collision>rear_bumper_collision</collision></contact>
+      </sensor>
+    </gazebo>
     <!-- Warm-white moulded nose and asymmetric equipment fairings.  The arm
          shoulder remains open above the right cowl. -->
@@ -97,5 +107,15 @@
       <xacro:hf_body_visual mesh="sensor_pylon_fairing.stl" material="sensor_pylon" rgba="0.070 0.085 0.088 1" visible="${visible}"/>
       <xacro:hf_body_visual mesh="sensor_pylon_service_hatch.stl" material="sensor_pylon_hatch" rgba="0.16 0.18 0.19 1" visible="${visible}"/>
-      <collision name="rear_shell_collision"><origin xyz="-0.285 0 0.495"/><geometry><box size="0.53 0.70 0.52"/></geometry></collision>
+      <!-- Panelized collision follows the shell walls and deliberately leaves
+           the robot-deposition aperture open; a solid cabinet-sized box would
+           make a visually open hopper physically unusable. -->
+      <collision name="rear_shell_rear_wall_collision"><origin xyz="-0.540 0 0.495"/><geometry><box size="0.045 0.70 0.52"/></geometry></collision>
+      <collision name="rear_shell_left_wall_collision"><origin xyz="-0.285 0.365 0.495"/><geometry><box size="0.53 0.045 0.52"/></geometry></collision>
+      <collision name="rear_shell_right_wall_collision"><origin xyz="-0.285 -0.365 0.495"/><geometry><box size="0.53 0.045 0.52"/></geometry></collision>
+      <collision name="rear_shell_lower_collision"><origin xyz="-0.285 0 0.350"/><geometry><box size="0.53 0.68 0.23"/></geometry></collision>
+      <collision name="rear_shell_roof_left_collision"><origin xyz="-0.285 0.310 0.735"/><geometry><box size="0.53 0.080 0.055"/></geometry></collision>
+      <collision name="rear_shell_roof_right_collision"><origin xyz="-0.285 -0.255 0.735"/><geometry><box size="0.53 0.180 0.055"/></geometry></collision>
+      <collision name="rear_shell_roof_front_collision"><origin xyz="-0.065 0.135 0.735"/><geometry><box size="0.090 0.270 0.055"/></geometry></collision>
+      <collision name="rear_shell_roof_rear_collision"><origin xyz="-0.500 0.135 0.735"/><geometry><box size="0.080 0.270 0.055"/></geometry></collision>
       <collision name="pylon_fairing_collision"><origin xyz="-0.135 0 0.770"/><geometry><box size="0.13 0.15 0.35"/></geometry></collision>
       <xacro:hf_bodywork_box_inertial mass="3.10" sx="0.55" sy="0.76" sz="0.58" xyz="-0.28 0 0.49"/>

File: starter_ws/src/sanitation_vehicle_description/urdf/high_fidelity/cleaning_mechanism.xacro (robot description, xacro)
@@ -315,5 +315,5 @@
       <xacro:hf_clean_visual mesh="suction_nozzle.stl"
         material="hf_nozzle" rgba="0.075 0.09 0.10 1"/>
-      <collision><geometry><box size="0.100 0.650 0.085"/></geometry></collision>
+      <collision name="suction_nozzle_link_collision"><geometry><box size="0.100 0.650 0.085"/></geometry></collision>
       <xacro:hf_cleaning_box_inertial mass="0.400" sx="0.100" sy="0.650" sz="0.085"/>
     </link>
@@ -322,4 +322,10 @@
       <origin xyz="0.040 0 0.010" rpy="0 0 0"/>
     </joint>
+    <gazebo reference="suction_nozzle_link">
+      <sensor name="suction_nozzle_ground_contact" type="contact">
+        <topic>/cleaning/suction_nozzle/contact</topic><update_rate>100</update_rate><always_on>true</always_on>
+        <contact><collision>suction_nozzle_link_collision</collision></contact>
+      </sensor>
+    </gazebo>
     <!-- Segmented hose geometry reserves a 50 mm ID flow path.  The three
          centres follow one continuous rising route from the rear nozzle into
@@ -371,4 +377,20 @@
       <origin xyz="-0.1075 0 0" rpy="0 ${pi/2.0} 0"/>
     </joint>
+    <!-- The externally observable motor/diaphragm drive is no longer a fixed
+         decorative pump.  This rotor joint is the controlled shaft datum used
+         by the recovery controller and hydraulic accounting layer. -->
+    <link name="recovery_pump_rotor_link">
+      <xacro:hf_clean_visual mesh="jabsco_pump_rotor.stl"
+        material="hf_pump_rotor" rgba="0.58 0.61 0.62 1"/>
+      <collision><geometry><cylinder radius="0.035" length="0.018"/></geometry></collision>
+      <xacro:hf_cleaning_cylinder_z_inertial mass="0.120" radius="0.035" length="0.018"/>
+    </link>
+    <joint name="recovery_pump_joint" type="continuous">
+      <parent link="recovery_pump_head_link"/><child link="recovery_pump_rotor_link"/>
+      <origin xyz="0 0 0.043" rpy="0 0 0"/>
+      <axis xyz="0 0 1"/>
+      <limit effort="18.0" velocity="62.832"/>
+      <dynamics damping="0.025" friction="0.015"/>
+    </joint>
     <link name="recovery_pump_isolator_mount_link">
       <xacro:hf_clean_visual mesh="pump_isolator_mount.stl"
@@ -391,4 +413,14 @@
       <origin xyz="0 -0.095 0" rpy="0 0 0"/>
     </joint>
+    <link name="recovery_flow_sensor_link">
+      <xacro:hf_clean_visual mesh="inline_flow_sensor.stl"
+        material="hf_flow_sensor" rgba="0.08 0.28 0.38 1"/>
+      <collision><geometry><box size="0.070 0.105 0.075"/></geometry></collision>
+      <xacro:hf_cleaning_box_inertial mass="0.220" sx="0.070" sy="0.105" sz="0.075"/>
+    </link>
+    <joint name="recovery_flow_sensor_mount_joint" type="fixed">
+      <parent link="wastewater_delivery_coupling_link"/><child link="recovery_flow_sensor_link"/>
+      <origin xyz="0 -0.095 0" rpy="0 0 0"/>
+    </joint>
   </xacro:macro>
 </robot>

File: starter_ws/src/sanitation_vehicle_description/urdf/high_fidelity/control_interfaces.xacro (robot description, xacro)
@@ -51,8 +51,10 @@
       <xacro:hf_velocity_joint name="right_side_brush_joint" max_velocity="31.416" max_effort="12.0"/>
       <xacro:hf_velocity_joint name="central_roller_joint" max_velocity="52.36" max_effort="20.0"/>
+      <xacro:hf_velocity_joint name="recovery_pump_joint" max_velocity="62.832" max_effort="18.0"/>
       <xacro:hf_position_joint name="cleaning_lift_joint" lower="0.0" upper="0.1" velocity="0.05" effort="1000.0" initial_position="0.1"/>
       <xacro:hf_position_joint name="squeegee_pitch_joint" lower="-0.2" upper="0.2" velocity="0.3" effort="120.0"/>
       <xacro:hf_position_joint name="squeegee_float_joint" lower="0.0" upper="0.035" velocity="0.08" effort="250.0" initial_position="0.035"/>
       <xacro:hf_position_joint name="dry_bin_lid_joint" lower="0.0" upper="1.75" velocity="0.5" effort="60.0"/>
+      <xacro:hf_position_joint name="dry_deposit_gate_joint" lower="0.0" upper="1.75" velocity="0.8" effort="22.0"/>
       <xacro:hf_position_joint name="wastewater_lid_joint" lower="0.0" upper="1.57" velocity="0.5" effort="45.0"/>
     </ros2_control>

File: starter_ws/src/sanitation_vehicle_description/urdf/high_fidelity/storage_system.xacro (robot description, xacro)
@@ -110,5 +110,8 @@
       <xacro:hf_storage_visual mesh="dry_bin_lid.stl"
         material="hf_dry_lid" rgba="0.055 0.12 0.085 1"/>
-      <collision><origin xyz="0.254 0 0"/><geometry><box size="0.508 0.391 0.010"/></geometry></collision>
+      <collision name="dry_lid_left_collision"><origin xyz="0.254 0.143 0"/><geometry><box size="0.508 0.105 0.010"/></geometry></collision>
+      <collision name="dry_lid_right_collision"><origin xyz="0.254 -0.143 0"/><geometry><box size="0.508 0.105 0.010"/></geometry></collision>
+      <collision name="dry_lid_rear_collision"><origin xyz="0.0895 0 0"/><geometry><box size="0.179 0.181 0.010"/></geometry></collision>
+      <collision name="dry_lid_front_collision"><origin xyz="0.4185 0 0"/><geometry><box size="0.179 0.181 0.010"/></geometry></collision>
       <xacro:hf_storage_box_inertial mass="0.750" sx="0.508" sy="0.391" sz="0.010" xyz="0.254 0 0"/>
     </link>
@@ -120,4 +123,61 @@
       <dynamics damping="1.5" friction="0.8"/>
     </joint>
+    <!-- Robot-only deposition port.  The main lid remains the human service
+         lid; the smaller powered gate lets the UR5e drop a 30 mm object
+         without opening the whole 40 L compartment. -->
+    <link name="dry_deposit_hopper_link">
+      <xacro:hf_storage_visual mesh="dry_deposit_hopper.stl"
+        material="hf_deposit_hopper" rgba="0.10 0.32 0.22 1"/>
+      <collision name="dry_deposit_hopper_front"><origin xyz="0.067 0 0" rpy="0 -0.42 0"/><geometry><box size="0.010 0.165 0.092"/></geometry></collision>
+      <collision name="dry_deposit_hopper_rear"><origin xyz="-0.067 0 0" rpy="0 0.42 0"/><geometry><box size="0.010 0.165 0.092"/></geometry></collision>
+      <collision name="dry_deposit_hopper_left"><origin xyz="0 0.057 0" rpy="0.36 0 0"/><geometry><box size="0.120 0.010 0.088"/></geometry></collision>
+      <collision name="dry_deposit_hopper_right"><origin xyz="0 -0.057 0" rpy="-0.36 0 0"/><geometry><box size="0.120 0.010 0.088"/></geometry></collision>
+      <xacro:hf_storage_box_inertial mass="0.240" sx="0.190" sy="0.165" sz="0.080"/>
+    </link>
+    <joint name="dry_deposit_hopper_mount_joint" type="fixed">
+      <parent link="dry_bin_lid_link"/><child link="dry_deposit_hopper_link"/>
+      <!-- Raise the robot port above the product roof.  The long chute below
+           preserves a continuous gravity path to the lid aperture. -->
+      <origin xyz="0.254 0 0.350" rpy="0 0 0"/>
+    </joint>
+    <link name="dry_deposit_gate_link">
+      <xacro:hf_storage_visual mesh="dry_deposit_gate.stl"
+        material="hf_deposit_gate" rgba="0.055 0.075 0.070 1"/>
+      <collision><origin xyz="0.092 0 0"/><geometry><box size="0.184 0.158 0.008"/></geometry></collision>
+      <xacro:hf_storage_box_inertial mass="0.180" sx="0.184" sy="0.158" sz="0.020" xyz="0.092 0 0"/>
+    </link>
+    <joint name="dry_deposit_gate_joint" type="revolute">
+      <parent link="dry_deposit_hopper_link"/><child link="dry_deposit_gate_link"/>
+      <origin xyz="-0.095 0 0.044" rpy="0 0 0"/>
+      <axis xyz="0 1 0"/>
+      <limit lower="0.0" upper="1.75" effort="22.0" velocity="0.8"/>
+      <dynamics damping="0.7" friction="0.25"/>
+    </joint>
+    <link name="dry_deposit_chute_link">
+      <xacro:hf_storage_visual mesh="dry_deposit_chute.stl"
+        material="hf_deposit_chute" rgba="0.20 0.48 0.32 1"/>
+      <collision name="dry_deposit_chute_collision"><geometry><box size="0.125 0.100 0.350"/></geometry></collision>
+      <xacro:hf_storage_box_inertial mass="0.320" sx="0.130" sy="0.105" sz="0.350"/>
+    </link>
+    <joint name="dry_deposit_chute_mount_joint" type="fixed">
+      <parent link="dry_deposit_hopper_link"/><child link="dry_deposit_chute_link"/>
+      <origin xyz="0 0 -0.180" rpy="0 0 0"/>
+    </joint>
+    <link name="dry_deposit_presence_sensor_link">
+      <xacro:hf_storage_visual mesh="dry_bin_level_sensor.stl"
+        material="hf_deposit_sensor" rgba="0.05 0.20 0.34 1"/>
+      <collision><geometry><box size="0.040 0.055 0.022"/></geometry></collision>
+      <xacro:hf_storage_box_inertial mass="0.045" sx="0.040" sy="0.055" sz="0.022"/>
+    </link>
+    <joint name="dry_deposit_presence_sensor_joint" type="fixed">
+      <parent link="dry_deposit_hopper_link"/><child link="dry_deposit_presence_sensor_link"/>
+      <origin xyz="0.088 0 0.015" rpy="0 0 0"/>
+    </joint>
+    <gazebo reference="dry_deposit_chute_link">
+      <sensor name="dry_deposit_contact" type="contact">
+        <topic>/storage/dry_deposit/contact</topic><update_rate>50</update_rate><always_on>true</always_on>
+        <contact><collision>dry_deposit_chute_collision</collision></contact>
+      </sensor>
+    </gazebo>
     <link name="dry_bin_latch_link">
       <xacro:hf_storage_visual mesh="dry_bin_latch.stl"

Commit message: fix(vehicle): synchronize formal model acceptance truth

File: reports/engineering/formal_competition_vehicle.urdf (robot description, URDF)
Before this commit: robot tzcup_formal_sanitation_vehicle, 131 links, 130 joints
Links:
- link bodywork_front_cowl_link: geometry collision box size=0.39 0.19 0.22; collision box size=0.405 0.40 0.10
- link bodywork_rear_shell_link: geometry collision box size=0.045 0.70 0.080; collision box size=0.045 0.70 0.52
- link dry_bin_payload_reserve_link: geometry visual box size=0.485 0.355 0.233
- link dry_deposit_chute_link: geometry collision box size=0.008 0.100 0.350; collision box size=0.008 0.100 0.350
Joints:
- joint squeegee_float_joint: origin xyz=-0.445 0 -0.011 rpy=0 0 0 -> xyz=-0.445 0 -0.051 rpy=0 0 0
- joint suction_nozzle_mount_joint: origin xyz=0.040 0 0.010 rpy=0 0 0 -> xyz=0.040 0 -0.005 rpy=0 0 0

File: starter_ws/src/sanitation_vehicle_description/urdf/formal_competition_vehicle.urdf.xacro (robot description, xacro)
@@ -9,4 +9,5 @@
   <xacro:include filename="high_fidelity/control_interfaces.xacro"/>
   <xacro:arg name="use_sim" default="true"/>
+  <xacro:arg name="controller_config_path" default=""/>
   <xacro:arg name="dry_load_mass_kg" default="0.0"/>
   <xacro:arg name="wastewater_load_mass_kg" default="0.0"/>
@@ -29,7 +30,14 @@
   <xacro:if value="$(arg use_sim)">
     <gazebo>
-      <plugin filename="gz_ros2_control-system" name="gz_ros2_control::GazeboSimROS2ControlPlugin">
-        <parameters>$(find sanitation_vehicle_description)/config/formal_vehicle_controllers.yaml</parameters>
-      </plugin>
+      <xacro:if value="${'$(arg controller_config_path)' != ''}">
+        <plugin filename="gz_ros2_control-system" name="gz_ros2_control::GazeboSimROS2ControlPlugin">
+          <parameters>$(arg controller_config_path)</parameters>
+        </plugin>
+      </xacro:if>
+      <xacro:unless value="${'$(arg controller_config_path)' != ''}">
+        <plugin filename="gz_ros2_control-system" name="gz_ros2_control::GazeboSimROS2ControlPlugin">
+          <parameters>$(find sanitation_vehicle_description)/config/formal_vehicle_controllers.yaml</parameters>
+        </plugin>
+      </xacro:unless>
       <plugin filename="libDynamicPayloadSystem.so" name="sanitation_gazebo_control::DynamicPayloadSystem">
         <dry_topic>/model/tzcup_formal_sanitation_vehicle/payload/dry_mass_kg</dry_topic>

File: starter_ws/src/sanitation_vehicle_description/urdf/high_fidelity/storage_system.xacro (robot description, xacro)
@@ -208,7 +208,7 @@
     </joint>
     <link name="dry_bin_payload_reserve_link">
-      <visual name="forty_litre_usable_envelope"><geometry><box size="0.485 0.355 0.232"/></geometry><material name="hf_dry_payload"><color rgba="0.65 0.48 0.18 0.16"/></material></visual>
+      <visual name="forty_litre_usable_envelope"><geometry><box size="0.485 0.355 0.233"/></geometry><material name="hf_dry_payload"><color rgba="0.65 0.48 0.18 0.16"/></material></visual>
       <!-- No collision: physically grasped 3 cm cubes supply shape and contact. -->
-      <xacro:hf_storage_box_inertial mass="${dry_payload_mass}" sx="0.485" sy="0.355" sz="0.232"/>
+      <xacro:hf_storage_box_inertial mass="${dry_payload_mass}" sx="0.485" sy="0.355" sz="0.233"/>
     </link>
     <joint name="dry_bin_payload_reserve_joint" type="fixed">

Commit message: Refresh DART lift snapshot

File: reports/engineering/formal_competition_vehicle.urdf (robot description, URDF)
Before this commit: robot tzcup_formal_sanitation_vehicle, 196 links, 195 joints
Joints:
- joint cleaning_lift_joint: limit lower=0.0 upper=0.100 effort=300.0 velocity=0.0048 -> lower=0.0 upper=0.10002 effort=300.0 velocity=0.0048
