Commit message: Close formal cleaning contact geometry gaps

File: reports/engineering/formal_competition_vehicle.urdf (robot description, URDF)
Before this commit: robot tzcup_formal_sanitation_vehicle, 196 links, 195 joints
Joints:
- joint left_side_brush_motor_mount_joint: origin xyz=0.385 0.545 0.0294 rpy=0 0 0 -> xyz=0.385 0.545 0.0244 rpy=0 0 0
- joint right_side_brush_motor_mount_joint: origin xyz=0.385 -0.545 0.0294 rpy=0 0 0 -> xyz=0.385 -0.545 0.0244 rpy=0 0 0

File: starter_ws/src/sanitation_vehicle_description/urdf/high_fidelity/cleaning_mechanism.xacro (robot description, xacro)
@@ -65,5 +65,5 @@
       <!-- At the 100 mm downstroke work pose, this installation height
            puts the conservative bristle-sweep collision tangent to z=0. -->
-      <origin xyz="0.385 ${lateral_sign * 0.545} 0.0294" rpy="0 0 0"/>
+      <origin xyz="0.385 ${lateral_sign * 0.545} 0.0244" rpy="0 0 0"/>
     </joint>
     <link name="${side}_side_brush_encoder_link">
@@ -448,9 +448,9 @@
       <plugin filename="libSqueegeeComplianceSystem.so"
               name="sanitation_gazebo_auxiliary::SqueegeeComplianceSystem">
-        <!-- -6 mm reference gives 10.8 N nominal preload at the ground-tangent
+        <!-- -6.5 mm reference gives 11.7 N nominal preload at the ground-tangent
              zero pose.  The contact solver supplies the opposing ground load. -->
         <float_stiffness_n_per_m>1800.0</float_stiffness_n_per_m>
         <float_damping_ns_per_m>45.0</float_damping_ns_per_m>
-        <float_preload_reference_m>-0.006</float_preload_reference_m>
+        <float_preload_reference_m>-0.0065</float_preload_reference_m>
         <float_max_force_n>120.0</float_max_force_n>
         <pitch_stiffness_nm_per_rad>32.0</pitch_stiffness_nm_per_rad>
